Commit message: updated all files

File: RBE594_ws/src/sirgas_description/urdf/gear_starter_motor.urdf.xacro (robot description, xacro)
@@ -29,11 +29,11 @@
         </inertial>
     </link>
-    <joint name="mh_gr_joint" type="revolute">
+    <joint name="mh_gr_joint" type="continuous">
         <parent link="motor_housing"/>
         <child link="gear_rotator"/>
-        <origin rpy="${pi} 0 0" xyz="0.0 0 0.05"/>
+        <origin rpy="${pi} 0 0" xyz="0.0 0 0.055"/>
         <axis xyz="0 0 1"/>
-        <limit effort="1500.0" lower="${-2*pi}" upper="${2*pi}" velocity="10.0"/>
-        <dynamics damping="0" friction="0"/>
+        <dynamics damping="1.0" friction="0.1"/>
+        <limit effort="1000.0" velocity="10.0"/>
     </joint>
     <link name="gear_rotator">
@@ -54,8 +54,28 @@
         </collision>
         <inertial>
-            <mass value="5.00"/>
+            <mass value="0.23"/>
             <origin rpy="0 0 0" xyz="0 0 0"/>
             <inertia ixx="0.0004399" ixy="0.0" ixz="0.0" iyx="0.0" iyy="0.0004399" iyz="0.0" izx="0.0" izy= "0.0" izz="0.00017253"/>
         </inertial>
     </link>
+    <!-- ROS2 Control Plugin-->
+    <ros2_control name="gsm_control" type="system">
+        <hardware>
+            <plugin>gz_ros2_control/GazeboSimSystem</plugin>
+        </hardware>
+        <joint name="mh_gr_joint">
+            <command_interface name="velocity">
+                <param name="min">-10</param>
+                <param name="max">10</param>
+            </command_interface>
+            <state_interface name="position"/>
+            <state_interface name="velocity"/>
+        </joint>
+    </ros2_control>
+    <!-- Fixed Ignition Gazebo plugin for ROS 2 Control -->
+    <gazebo>
+        <plugin filename="libgz_ros2_control-system.so" name="gz_ros2_control::GazeboSimROS2ControlPlugin">
+            <parameters>$(find sirgas_description)/config/gsm_controller.yaml</parameters>
+        </plugin>
+    </gazebo>
 </robot>

File: RBE594_ws/src/sirgas_description/urdf/pba.urdf.xacro (robot description, xacro)
@@ -166,16 +166,20 @@
             <state_interface name="position"/>
             <state_interface name="velocity"/>
+            <state_interface name="effort"/>
         </joint>
         <joint name="pb_first_joint">
             <state_interface name="position"/>
             <state_interface name="velocity"/>
+            <state_interface name="effort"/>
         </joint>
         <joint name="pb_second_joint">
             <state_interface name="position"/>
             <state_interface name="velocity"/>
+            <state_interface name="effort"/>
         </joint>
         <joint name="pb_third_joint">
             <state_interface name="position"/>
             <state_interface name="velocity"/>
+            <state_interface name="effort"/>
         </joint>
     </ros2_control>
@@ -183,4 +187,5 @@
         <plugin filename="libgz_ros2_control-system.so" name="gz_ros2_control::GazeboSimROS2ControlPlugin">
             <parameters>$(find sirgas_description)/config/pba_controller.yaml</parameters>
+            <controller_manager_name>pba_controller_manager</controller_manager_name>
         </plugin>
     </gazebo>

File: RBE594_ws/src/sirgas_description/urdf/ur20.ros2_control.xacro (robot description, xacro)
@@ -3,6 +3,7 @@
   <xacro:macro name="ur_ros2_control" params="
     name
-    use_fake_hardware:=false fake_sensor_commands:=false
-    sim_gazebo:=false
+    use_fake_hardware:=false
+    fake_sensor_commands:=false
+    sim_gazebo:=true
     sim_ignition:=false
     headless_mode:=false
@@ -21,12 +22,9 @@
     non_blocking_read:=true
     keep_alive_count:=2
-    ">
+">
     <ros2_control name="${name}" type="system">
       <hardware>
-        <xacro:if value="${sim_gazebo}">
-          <plugin>gazebo_ros2_control/GazeboSystem</plugin>
-        </xacro:if>
-        <xacro:if value="${sim_ignition}">
-          <plugin>ign_ros2_control/IgnitionSystem</plugin>
+        <xacro:if value="${(sim_gazebo or sim_ignition) and not use_fake_hardware}">
+          <plugin>gz_ros2_control/GazeboSimSystem</plugin>
         </xacro:if>
         <xacro:if value="${use_fake_hardware}">
@@ -42,5 +40,5 @@
           <param name="output_recipe_filename">${output_recipe_filename}</param>
           <param name="input_recipe_filename">${input_recipe_filename}</param>
-          <param name="headless_mode">${headless_mode}</param>
+       <param name="headless_mode">${headless_mode}</param>
           <param name="reverse_port">${reverse_port}</param>
           <param name="script_sender_port">${script_sender_port}</param>
@@ -69,5 +67,4 @@
         <command_interface name="velocity"/>
         <state_interface name="position">
-          <!-- initial position for the FakeSystem and simulation -->
           <param name="initial_value">${initial_positions['shoulder_pan_joint']}</param>
         </state_interface>
@@ -79,7 +76,6 @@
         <command_interface name="velocity"/>
         <state_interface name="position">
-          <!-- initial position for the FakeSystem and simulation -->
           <param name="initial_value">${initial_positions['shoulder_lift_joint']}</param>
-        </state_interface>
+          </state_interface>
         <state_interface name="velocity"/>
         <state_interface name="effort"/>
@@ -89,5 +85,4 @@
         <command_interface name="velocity"/>
         <state_interface name="position">
-          <!-- initial position for the FakeSystem and simulation -->
           <param name="initial_value">${initial_positions['elbow_joint']}</param>
         </state_interface>
@@ -99,8 +94,7 @@
         <command_interface name="velocity"/>
         <state_interface name="position">
-          <!-- initial position for the FakeSystem and simulation -->
           <param name="initial_value">${initial_positions['wrist_1_joint']}</param>
         </state_interface>
-        <state_interface name="velocity"/>
+          <state_interface name="velocity"/>
         <state_interface name="effort"/>
       </joint>
@@ -109,9 +103,8 @@
         <command_interface name="velocity"/>
         <state_interface name="position">
-          <!-- initial position for the FakeSystem and simulation -->
           <param name="initial_value">${initial_positions['wrist_2_joint']}</param>
         </state_interface>
         <state_interface name="velocity"/>
-        <state_interface name="effort"/>
+          <state_interface name="effort"/>
       </joint>
       <joint name="${tf_prefix}wrist_3_joint">
@@ -119,9 +112,8 @@
         <command_interface name="velocity"/>
         <state_interface name="position">
-          <!-- initial position for the FakeSystem and simulation -->
           <param name="initial_value">${initial_positions['wrist_3_joint']}</param>
         </state_interface>
         <state_interface name="velocity"/>
-        <state_interface name="effort"/>
+          <state_interface name="effort"/>
       </joint>
       <xacro:unless value="${sim_gazebo or sim_ignition}">
@@ -133,5 +125,5 @@
           <state_interface name="torque.y"/>
           <state_interface name="torque.z"/>
-        </sensor>
+          </sensor>
         <sensor name="${tf_prefix}tcp_pose">
           <state_interface name="position.x"/>
@@ -143,6 +135,5 @@
           <state_interface name="orientation.w"/>
         </sensor>
-        <!-- NOTE The following are joints used only for testing with fake hardware and will change in the future -->
-        <gpio name="${tf_prefix}speed_scaling">
+          <gpio name="${tf_prefix}speed_scaling">
           <state_interface name="speed_scaling_factor"/>
           <param name="initial_speed_scaling_factor">1</param>
@@ -169,5 +160,6 @@
           <command_interface name="standard_digital_output_cmd_16"/>
           <command_interface name="standard_digital_output_cmd_17"/>
-          <command_interface name="standard_analog_output_cmd_0"/>
+          <command_interface
+          name="standard_analog_output_cmd_0"/>
           <command_interface name="standard_analog_output_cmd_1"/>
           <command_interface name="analog_output_domain_cmd"/>
@@ -252,5 +244,5 @@
           <command_interface name="payload_async_success"/>
         </gpio>
-        <gpio name="${tf_prefix}resend_robot_program">
+          <gpio name="${tf_prefix}resend_robot_program">
           <command_interface name="resend_robot_program_cmd"/>
           <command_interface name="resend_robot_program_async_success"/>
@@ -283,5 +275,5 @@
         <command_interface name="task_frame_rx"/>
         <command_interface name="task_frame_ry"/>
-        <command_interface name="task_frame_rz"/>
+          <command_interface name="task_frame_rz"/>
         <command_interface name="selection_vector_x"/>
         <command_interface name="selection_vector_y"/>
@@ -294,5 +286,5 @@
         <command_interface name="wrench_z"/>
         <command_interface name="wrench_rx"/>
-        <command_interface name="wrench_ry"/>
+          <command_interface name="wrench_ry"/>
         <command_interface name="wrench_rz"/>
         <command_interface name="limits_x"/>
@@ -305,5 +297,6 @@
         <command_interface name="damping"/>
         <command_interface name="gain_scaling"/>
-        <command_interface name="disable_cmd"/>
+        <command_interface
+          name="disable_cmd"/>
         <command_interface name="force_mode_async_success"/>
       </gpio>
@@ -317,5 +310,5 @@
         <command_interface name="setpoint_velocities_0"/>
         <command_interface name="setpoint_velocities_1"/>
-        <command_interface name="setpoint_velocities_2"/>
+          <command_interface name="setpoint_velocities_2"/>
         <command_interface name="setpoint_velocities_3"/>
         <command_interface name="setpoint_velocities_4"/>
@@ -328,5 +321,5 @@
         <command_interface name="setpoint_accelerations_5"/>
         <command_interface name="transfer_state"/>
-        <command_interface name="time_from_start"/>
+          <command_interface name="time_from_start"/>
         <command_interface name="abort"/>
       </gpio>

File: RBE594_ws/src/sirgas_description/urdf/ur20_macro.xacro (robot description, xacro)
@@ -1,6 +1,6 @@
 <?xml version="1.0"?>
 <robot xmlns:xacro="http://wiki.ros.org/xacro">
-  <xacro:include filename="$(find ur_description)/urdf/inc/ur_transmissions.xacro" />
-  <xacro:include filename="$(find ur_description)/urdf/inc/ur_common.xacro" />
+  <xacro:include filename="$(find sirgas_description)/urdf/inc/ur_transmissions.xacro" />
+  <xacro:include filename="$(find sirgas_description)/urdf/inc/ur_common.xacro" />
   <xacro:macro name="ur_robot" params="
     name
@@ -19,5 +19,5 @@
     use_fake_hardware:=false
     fake_sensor_commands:=false
-    sim_gazebo:=false
+    sim_gazebo:=true
     sim_ignition:=false
     headless_mode:=false

File: RBE594_ws/src/sirgas_description/urdf/ur20_picker.urdf.xacro (robot description, xacro)
@@ -1,13 +1,8 @@
 <?xml version="1.0"?>
-<robot xmlns:xacro="http://wiki.ros.org/xacro" name="ur">
-   <!-- robot name parameter -->
-   <xacro:arg name="name" default="ur"/>
-   <!-- import main macro -->
+<robot xmlns:xacro="http://wiki.ros.org/xacro" name="ur20_picker">
+   <xacro:arg name="name" default="ur20_picker"/>
    <xacro:include filename="$(find sirgas_description)/urdf/ur20_macro.xacro"/>
-   <!-- possible 'ur_type' values: ur3, ur5, ur10, ur3e, ur5e, ur7e, ur10e, ur12e, ur16e, ur8long, ur15, ur20, ur30 -->
-   <!-- the default value should raise an error in case this was called without defining the type -->
    <xacro:arg name="ur_type" default="ur20"/>
-   <!-- parameters -->
-   <xacro:arg name="tf_prefix" default="" />
+   <xacro:arg name="tf_prefix" default="ur20_picker/" />
    <xacro:arg name="joint_limit_params" default="$(find ur_description)/config/$(arg ur_type)/joint_limits.yaml"/>
    <xacro:arg name="kinematics_params" default="$(find ur_description)/config/$(arg ur_type)/default_kinematics.yaml"/>
@@ -18,5 +13,4 @@
    <xacro:arg name="safety_pos_margin" default="0.15"/>
    <xacro:arg name="safety_k_position" default="20"/>
-   <!-- ros2_control related parameters -->
    <xacro:arg name="headless_mode" default="false" />
    <xacro:arg name="robot_ip" default="0.0.0.0" />
@@ -29,5 +23,4 @@
    <xacro:arg name="script_sender_port" default="50002"/>
    <xacro:arg name="trajectory_port" default="50003"/>
-   <!--   tool communication related parameters-->
    <xacro:arg name="use_tool_communication" default="false" />
    <xacro:arg name="tool_voltage" default="0" />
@@ -39,43 +32,16 @@
    <xacro:arg name="tool_device_name" default="/tmp/ttyUR" />
    <xacro:arg name="tool_tcp_port" default="54321" />
-     <!-- Simulation parameters -->
    <xacro:arg name="use_fake_hardware" default="false" />
    <xacro:arg name="fake_sensor_commands" default="false" />
    <xacro:arg name="sim_gazebo" default="true" />
    <xacro:arg name="sim_ignition" default="false" />
-   <xacro:arg name="simulation_controllers" default="$(find sirgas_description)/config/ur20_controllers.yaml" />
-   <!-- initial position for simulations (Fake Hardware, Gazebo, Ignition) -->
+   <xacro:arg name="simulation_controllers" default="$(find sirgas_description)/config/ur20_picker_controllers.yaml" />
    <xacro:arg name="initial_positions_file" default="$(find sirgas_description)/config/initial_positions.yaml"/>
-   <!-- convert to property to use substitution in function -->
    <xacro:property name="initial_positions_file" default="$(arg initial_positions_file)"/>
    <xacro:property name="is_sim_gazebo" value="$(arg sim_gazebo)"/>
    <xacro:property name="is_sim_ignition" value="$(arg sim_ignition)"/>
-   <!-- create link fixed to the "world" -->
-   <link name="world" />
-   <xacro:if value="${is_sim_gazebo or is_sim_ignition}">
-     <link name="ground_plane">
-       <visual>
-         <origin rpy="0 0 0" xyz="0 0 0"/>
-         <geometry>
-           <box size="5 5 0"/>
-         </geometry>
-         <material name="ground_white">
-           <color rgba="1 1 1 0.5"/>
-         </material>
-       </visual>
-       <collision>
-         <origin rpy="0 0 0" xyz="0 0 0"/>
-         <geometry>
-           <box size="5 5 0"/>
-         </geometry>
-       </collision>
-     </link>
-     <joint name="ground_plane_joint" type="fixed">
-       <origin xyz="0 0 -0.01" rpy="0 0 0"/>
-       <parent link="world"/>
-       <child link="ground_plane"/>
-     </joint>
-   </xacro:if>
-   <!-- arm -->
+   <xacro:property name="is_fake_hardware" value="$(arg use_fake_hardware)"/>
+   <!-- Define a minimal world link for the URDF to be valid -->
+   <link name="world"/>
    <xacro:ur_robot
      name="$(arg name)"
@@ -115,26 +81,26 @@
      trajectory_port="$(arg trajectory_port)"
      >
-     <origin xyz="0 0 0" rpy="0 0 0" />          <!-- position robot in the world -->
+     <origin xyz="0.5 -0.5 0.0" rpy="0 0 0" />  <!-- Position in world -->
    </xacro:ur_robot>
-   <xacro:if value="$(arg sim_gazebo)">
-    <!-- Gazebo plugins -->
-    <gazebo reference="world">
-    </gazebo>
-    <gazebo>
-      <plugin filename="libgazebo_ros2_control.so" name="gazebo_ros2_control">
-        <parameters>$(arg simulation_controllers)</parameters>
-      </plugin>
-    </gazebo>
-  </xacro:if>
-  <xacro:if value="$(arg sim_ignition)">
-    <!-- Gazebo plugins -->
-    <gazebo reference="world">
-    </gazebo>
-    <gazebo>
-      <plugin filename="libign_ros2_control-system.so" name="ign_ros2_control::IgnitionROS2ControlPlugin">
-        <parameters>$(arg simulation_controllers)</parameters>
-        <controller_manager_node_name>$(arg tf_prefix)controller_manager</controller_manager_node_name>
-      </plugin>
-    </gazebo>
-  </xacro:if>
+   <!-- Gazebo plugins - only add if this is the main robot in simulation -->
+   <xacro:if value="${is_sim_gazebo and not is_fake_hardware}">
+     <gazebo>
+       <plugin filename="libgazebo_ros2_control.so" name="gazebo_ros2_control">
+         <parameters>$(arg simulation_controllers)</parameters>
+         <controller_manager_name>$(arg name)_controller_manager</controller_manager_name>
+         <robot_param>/$(arg name)/robot_description</robot_param>
+         <robot_param_node>$(arg name)_robot_state_publisher</robot_param_node>
+       </plugin>
+     </gazebo>
+   </xacro:if>
+   <xacro:if value="${is_sim_ignition}">
+     <gazebo>
+       <plugin filename="libign_ros2_control-system.so" name="ign_ros2_control::IgnitionSystem">
+         <parameters>$(arg simulation_controllers)</parameters>
+         <controller_manager_name>$(arg name)_controller_manager</controller_manager_name>
+         <robot_param>/$(arg name)/robot_description</robot_param>
+         <robot_param_node>$(arg name)_robot_state_publisher</robot_param_node>
+       </plugin>
+     </gazebo>
+   </xacro:if>
 </robot>

File: RBE594_ws/src/sirgas_description/urdf/ur20_starter.urdf.xacro (robot description, xacro)
@@ -1,13 +1,8 @@
 <?xml version="1.0"?>
-<robot xmlns:xacro="http://wiki.ros.org/xacro" name="ur">
-   <!-- robot name parameter -->
-   <xacro:arg name="name" default="ur"/>
-   <!-- import main macro -->
+<robot xmlns:xacro="http://wiki.ros.org/xacro" name="$ur20_starter">
+   <xacro:arg name="name" default="ur20_starter"/>
    <xacro:include filename="$(find sirgas_description)/urdf/ur20_macro.xacro"/>
-   <!-- possible 'ur_type' values: ur3, ur5, ur10, ur3e, ur5e, ur7e, ur10e, ur12e, ur16e, ur8long, ur15, ur20, ur30 -->
-   <!-- the default value should raise an error in case this was called without defining the type -->
    <xacro:arg name="ur_type" default="ur20"/>
-   <!-- parameters -->
-   <xacro:arg name="tf_prefix" default="" />
+   <xacro:arg name="tf_prefix" default="ur20_starter/" />
    <xacro:arg name="joint_limit_params" default="$(find ur_description)/config/$(arg ur_type)/joint_limits.yaml"/>
    <xacro:arg name="kinematics_params" default="$(find ur_description)/config/$(arg ur_type)/default_kinematics.yaml"/>
@@ -18,5 +13,4 @@
    <xacro:arg name="safety_pos_margin" default="0.15"/>
    <xacro:arg name="safety_k_position" default="20"/>
-   <!-- ros2_control related parameters -->
    <xacro:arg name="headless_mode" default="false" />
    <xacro:arg name="robot_ip" default="0.0.0.0" />
@@ -29,5 +23,4 @@
    <xacro:arg name="script_sender_port" default="50002"/>
    <xacro:arg name="trajectory_port" default="50003"/>
-   <!--   tool communication related parameters-->
    <xacro:arg name="use_tool_communication" default="false" />
    <xacro:arg name="tool_voltage" default="0" />
@@ -39,43 +32,16 @@
    <xacro:arg name="tool_device_name" default="/tmp/ttyUR" />
    <xacro:arg name="tool_tcp_port" default="54321" />
-     <!-- Simulation parameters -->
    <xacro:arg name="use_fake_hardware" default="false" />
    <xacro:arg name="fake_sensor_commands" default="false" />
-   <xacro:arg name="sim_gazebo" default="false" />
+   <xacro:arg name="sim_gazebo" default="true" />
    <xacro:arg name="sim_ignition" default="false" />
-   <xacro:arg name="simulation_controllers" default="$(find sirgas_description)/config/ur20_controllers.yaml" />
-   <!-- initial position for simulations (Fake Hardware, Gazebo, Ignition) -->
+   <xacro:arg name="simulation_controllers" default="$(find sirgas_description)/config/ur20_starter_controllers.yaml" />
    <xacro:arg name="initial_positions_file" default="$(find sirgas_description)/config/initial_positions.yaml"/>
-   <!-- convert to property to use substitution in function -->
    <xacro:property name="initial_positions_file" default="$(arg initial_positions_file)"/>
    <xacro:property name="is_sim_gazebo" value="$(arg sim_gazebo)"/>
    <xacro:property name="is_sim_ignition" value="$(arg sim_ignition)"/>
-   <!-- create link fixed to the "world" -->
-   <link name="world" />
-   <xacro:if value="${is_sim_gazebo or is_sim_ignition}">
-     <link name="ground_plane">
-       <visual>
-         <origin rpy="0 0 0" xyz="0 0 0"/>
-         <geometry>
-           <box size="5 5 0"/>
-         </geometry>
-         <material name="ground_white">
-           <color rgba="1 1 1 0.5"/>
-         </material>
-       </visual>
-       <collision>
-         <origin rpy="0 0 0" xyz="0 0 0"/>
-         <geometry>
-           <box size="5 5 0"/>
-         </geometry>
-       </collision>
-     </link>
-     <joint name="ground_plane_joint" type="fixed">
-       <origin xyz="0 0 -0.01" rpy="0 0 0"/>
-       <parent link="world"/>
-       <child link="ground_plane"/>
-     </joint>
-   </xacro:if>
-   <!-- arm -->
+   <xacro:property name="is_fake_hardware" value="$(arg use_fake_hardware)"/>
+   <!-- Define a minimal world link for the URDF to be valid -->
+   <link name="world"/>
    <xacro:ur_robot
      name="$(arg name)"
@@ -115,26 +81,24 @@
      trajectory_port="$(arg trajectory_port)"
      >
-     <origin xyz="0 0 0" rpy="0 0 0" />          <!-- position robot in the world -->
+     <origin xyz="0.0 0.0 0.0" rpy="0 0 0" />  <!-- Position in world -->
    </xacro:ur_robot>
-   <xacro:if value="$(arg sim_gazebo)">
-    <!-- Gazebo plugins -->
-    <gazebo reference="world">
+   <!-- Gazebo plugins - only add if this is the main robot in simulation -->
+   <xacro:if value="${is_sim_gazebo and not is_fake_hardware}">
+     <gazebo>
+        <plugin filename="libgz_ros2_control-system.so" name="gz_ros2_control::GazeboSimROS2ControlPlugin">
+            <parameters>$(arg simulation_controllers)</parameters>
+            <controller_manager_name>$(arg name)_controller_manager</controller_manager_name>
+            <robot_param>/$(arg name)/robot_description</robot_param>
+            <ros2_control_names>$(arg name)</ros2_control_names>
+        </plugin>
     </gazebo>
-    <gazebo>
-      <plugin filename="libgazebo_ros2_control.so" name="gazebo_ros2_control">
-        <parameters>$(arg simulation_controllers)</parameters>
-      </plugin>
-    </gazebo>
-  </xacro:if>
-  <xacro:if value="$(arg sim_ignition)">
-    <!-- Gazebo plugins -->
-    <gazebo reference="world">
-    </gazebo>
-    <gazebo>
-      <plugin filename="libign_ros2_control-system.so" name="ign_ros2_control::IgnitionROS2ControlPlugin">
-        <parameters>$(arg simulation_controllers)</parameters>
-        <controller_manager_node_name>$(arg tf_prefix)controller_manager</controller_manager_node_name>
-      </plugin>
-    </gazebo>
-  </xacro:if>
+   </xacro:if>
+   <xacro:if value="${is_sim_ignition}">
+     <gazebo>
+       <plugin filename="libgz_ros2_control-system.so" name="gz_ros2_control::GazeboSimROS2ControlPlugin">
+         <parameters>$(arg simulation_controllers)</parameters>
+         <controller_manager_name>$(arg name)_controller_manager</controller_manager_name>
+         </plugin>
+     </gazebo>
+   </xacro:if>
 </robot>
