Commit message: Added files for gripper attachment

File: RBE594_ws/src/sirgas_description/urdf/ur20_pba.urdf.xacro (robot description, xacro)
@@ -7,3 +7,50 @@
     <!-- Import PBA Robot - directly include without macro call -->
     <xacro:include filename="$(find sirgas_description)/urdf/pba2.urdf.xacro" />
+    <!-- Import UR20 Gripper Robot - directly include without macro call -->
+    <xacro:include filename="$(find sirgas_description)/urdf/robotiq_arg85_description.urdf.xacro" />
+    <joint name="wrist3_gripper_joint" type="continuous">
+        <parent link="ur20_starter/wrist_3_link"/>
+        <child link="robotiq_85_base_link"/>
+        <origin rpy="0 0 0" xyz="0 0 0"/>
+        <axis xyz="0 0 1"/>
+        <limit effort="1500.0" velocity="10.0"/>
+        <dynamics damping="0.1" friction="0.01"/>
+    </joint>
+     <!-- Add ROS2 Control for Gripper -->
+    <ros2_control name="gripper_controller" type="system">
+        <hardware>
+            <plugin>gz_ros2_control/GazeboSimSystem</plugin>
+        </hardware>
+        <joint name="finger_joint">
+            <command_interface name="position"/>
+            <state_interface name="position"/>
+            <state_interface name="velocity"/>
+            <state_interface name="effort"/>
+        </joint>
+        <joint name="left_inner_knuckle_joint">
+            <state_interface name="position"/>
+            <state_interface name="velocity"/>
+            <state_interface name="effort"/>
+        </joint>
+        <joint name="left_inner_finger_joint">
+            <state_interface name="position"/>
+            <state_interface name="velocity"/>
+            <state_interface name="effort"/>
+        </joint>
+        <joint name="right_inner_knuckle_joint">
+            <state_interface name="position"/>
+            <state_interface name="velocity"/>
+            <state_interface name="effort"/>
+        </joint>
+        <joint name="right_inner_finger_joint">
+            <state_interface name="position"/>
+            <state_interface name="velocity"/>
+            <state_interface name="effort"/>
+        </joint>
+        <joint name="right_outer_knuckle_joint">
+            <state_interface name="position"/>
+            <state_interface name="velocity"/>
+            <state_interface name="effort"/>
+        </joint>
+    </ros2_control>
 </robot>
