Commit message: fixing master

File: RBE594_ws/src/sirgas_description/urdf/panda.urdf.xacro (robot description, xacro)
@@ -6,5 +6,5 @@
 <robot name="panda" xmlns:xacro="http://www.ros.org/wiki/xacro">
     <joint name="world_link0_joint" type="fixed">
-        <origin rpy="0 0 0" xyz="0 0.5 0" />
+        <origin rpy="0 0 0" xyz="0 -0.5 0" />
         <parent link="world" />
         <child link="panda_link0" />

File: RBE594_ws/src/sirgas_description/urdf/pba2.urdf.xacro (robot description, xacro)
@@ -93,7 +93,7 @@
         parent_link="first_gear"
         tag_size=".5"
-        tag_thickness="0.002"
+        tag_thickness="0.00001"
         xyz="0 .06 1.0"
-        rpy="0 3.14 0"
+        rpy="0 3.0 0"
         link_name="first_gear_apriltag"
     />
