Commit message: updated all files. Best working launch file is sim6.launch.py as that one launches the panda robot with all working controllers and a semi-working MoveIt configuration

File: RBE594_ws/src/sirgas_description/urdf/pba2.urdf.xacro (robot description, xacro)
@@ -154,5 +154,5 @@
      <!-- Only the master joint (pb_starter_joint) gets command interfaces -->
      <!-- Mimic joints only get state interfaces -->
-    <ros2_control name="combined_controller" type="system">
+    <!-- <ros2_control name="combined_controller" type="system">
         <hardware>
             <plugin>gz_ros2_control/GazeboSimSystem</plugin>
@@ -188,4 +188,4 @@
             <controller_manager_name>combined_controller_manager</controller_manager_name>
         </plugin>
-    </gazebo>
+    </gazebo> -->
 </robot>

File: RBE594_ws/src/sirgas_description/urdf/ur20_pba.urdf.xacro (robot description, xacro)
@@ -9,11 +9,8 @@
     <!-- Import UR20 Gripper Robot - directly include without macro call -->
     <xacro:include filename="$(find sirgas_description)/urdf/robotiq_arg85_description.urdf.xacro" />
-    <joint name="wrist3_gripper_joint" type="continuous">
-        <parent link="ur20_starter/wrist_3_link"/>
+    <joint name="tool0_gripper_joint" type="fixed">
+        <parent link="ur20_starter/tool0"/>
         <child link="robotiq_85_base_link"/>
         <origin rpy="0 0 0" xyz="0 0 0"/>
-        <axis xyz="0 0 1"/>
-        <limit effort="1500.0" velocity="10.0"/>
-        <dynamics damping="0.1" friction="0.01"/>
     </joint>
      <!-- Add ROS2 Control for Gripper -->

Commit message: fixing urdf

File: RBE594_ws/src/sirgas_description/urdf/pba2.urdf.xacro (robot description, xacro)
@@ -160,4 +160,141 @@
         </inertial>
     </link>
+    <!-- ==================== LINER LINKS AND JOINTS ==================== -->
+    <!-- Liner 1 -->
+    <link name="liner1">
+    <visual>
+        <origin xyz="0 0 0" rpy="0 0 0"/>
+        <geometry>
+        <box size="0.005 0.005 0.001"/>
+        </geometry>
+        <material name="Red">
+        <color rgba="1.0 0.0 0.0 1.0"/>
+        </material>
+    </visual>
+    </link>
+    <joint name="liner1_pbs" type="fixed">
+    <parent link="peg_board"/>
+    <child link="liner1"/>
+    <origin xyz="-0.375 -0.02225 0.176" rpy="0 0 0"/>
+    </joint>
+    <!-- Liner 2 -->
+    <link name="liner2">
+    <visual>
+        <origin xyz="0 0 0" rpy="0 0 0"/>
+        <geometry>
+        <box size="0.005 0.005 0.001"/>
+        </geometry>
+        <material name="Red">
+        <color rgba="1.0 0.0 0.0 1.0"/>
+        </material>
+    </visual>
+    </link>
+    <joint name="liner2_pbs" type="fixed">
+    <parent link="starter_gear"/>
+    <child link="liner2"/>
+    <origin xyz="0.0 -0.028 0.051" rpy="0 0 0"/>
+    </joint>
+    <!-- Liner 3 -->
+    <link name="liner3">
+    <visual>
+        <origin xyz="0 0 0" rpy="0 0 0"/>
+        <geometry>
+        <box size="0.005 0.005 0.001"/>
+        </geometry>
+        <material name="Red">
+        <color rgba="1.0 0.0 0.0 1.0"/>
+        </material>
+    </visual>
+    </link>
+    <joint name="liner3_pbf" type="fixed">
+    <parent link="peg_board"/>
+    <child link="liner3"/>
+    <origin xyz="0.0 -0.02225 0.176" rpy="0 0 0"/>
+    </joint>
+    <!-- Liner 4 -->
+    <link name="liner4">
+    <visual>
+        <origin xyz="0 0 0" rpy="0 0 0"/>
+        <geometry>
+        <box size="0.005 0.005 0.001"/>
+        </geometry>
+        <material name="Red">
+        <color rgba="1.0 0.0 0.0 1.0"/>
+        </material>
+    </visual>
+    </link>
+    <joint name="liner4_pbf" type="fixed">
+    <parent link="first_gear"/>
+    <child link="liner4"/>
+    <origin xyz="0.0 -0.028 0.051" rpy="0 0 0"/>
+    </joint>
+    <!-- Liner 5 -->
+    <link name="liner5">
+    <visual>
+        <origin xyz="0 0 0" rpy="0 0 0"/>
+        <geometry>
+        <box size="0.005 0.005 0.001"/>
+        </geometry>
+        <material name="Red">
+        <color rgba="1.0 0.0 0.0 1.0"/>
+        </material>
+    </visual>
+    </link>
+    <joint name="liner5_pbf" type="fixed">
+    <parent link="peg_board"/>
+    <child link="liner5"/>
+    <origin xyz="0.25 -0.02225 0.176" rpy="0 0 0"/>
+    </joint>
+    <!-- Liner 6 -->
+    <link name="liner6">
+    <visual>
+        <origin xyz="0 0 0" rpy="0 0 0"/>
+        <geometry>
+        <box size="0.005 0.005 0.001"/>
+        </geometry>
+        <material name="Red">
+        <color rgba="1.0 0.0 0.0 1.0"/>
+        </material>
+    </visual>
+    </link>
+    <joint name="liner6_pb2" type="fixed">
+    <parent link="second_gear"/>
+    <child link="liner6"/>
+    <origin xyz="0.0 -0.028 0.051" rpy="0 0 0"/>
+    </joint>
+    <!-- Liner 7 -->
+    <link name="liner7">
+    <visual>
+        <origin xyz="0 0 0" rpy="0 0 0"/>
+        <geometry>
+        <box size="0.005 0.005 0.001"/>
+        </geometry>
+        <material name="Red">
+        <color rgba="1.0 0.0 0.0 1.0"/>
+        </material>
+    </visual>
+    </link>
+    <joint name="liner7_pbt" type="fixed">
+    <parent link="peg_board"/>
+    <child link="liner7"/>
+    <origin xyz="0.45 -0.02225 0.176" rpy="0 0 0"/>
+    </joint>
+    <!-- Liner 8 -->
+    <link name="liner8">
+    <visual>
+        <origin xyz="0 0 0" rpy="0 0 0"/>
+        <geometry>
+        <box size="0.005 0.005 0.001"/>
+        </geometry>
+        <material name="Red">
+        <color rgba="1.0 0.0 0.0 1.0"/>
+        </material>
+    </visual>
+    </link>
+    <joint name="liner8_pbt" type="fixed">
+    <parent link="third_gear"/>
+    <child link="liner8"/>
+    <origin xyz="0.0 -0.028 0.051" rpy="0 0 0"/>
+    </joint>
      <!-- ROS 2 Control configuration -->
      <!-- Only the master joint (pb_starter_joint) gets command interfaces -->
