Commit message: Separated gears from peg_board

File: RBE594_ws/src/sirgas_description/urdf/cube.urdf.xacro (robot description, xacro)
@@ -6,9 +6,9 @@
         <color rgba="0.0 0.0 1.0 1.0" />
     </material>
-    <joint name="cube_world_joint" type="fixed">
+    <!-- <joint name="cube_world_joint" type="floating">
         <parent link="world"/>
         <child link="cube_link"/>
         <origin rpy="0 0 0" xyz="0 -1.0 ${cube_size/2}"/>
-    </joint>
+    </joint> -->
     <link name="cube_link">
         <visual>

File: RBE594_ws/src/sirgas_description/urdf/panda_pba.urdf.xacro (robot description, xacro)
@@ -6,5 +6,5 @@
     <xacro:include filename="$(find sirgas_description)/urdf/panda.urdf.xacro" />
     <!-- Import PBA Robot - directly include without macro call -->
-    <xacro:include filename="$(find sirgas_description)/urdf/pba2.urdf.xacro" />
+    <xacro:include filename="$(find sirgas_description)/urdf/pba.urdf.xacro" />
     <!-- Import PBA Robot - directly include without macro call -->
     <xacro:include filename="$(find sirgas_description)/urdf/camera2.urdf.xacro" />
@@ -62,5 +62,5 @@
         </joint>
         <!-- PBA Robot -->
-        <joint name="pb_starter_joint">
+        <!-- <joint name="pb_starter_joint">
             <command_interface name="velocity">
                 <param name="min">-10</param>
@@ -85,5 +85,5 @@
             <state_interface name="velocity"/>
             <state_interface name="effort"/>
-        </joint>
+        </joint> -->
     </ros2_control>
     <gazebo>

File: RBE594_ws/src/sirgas_description/urdf/pba.urdf.xacro (robot description, xacro)
@@ -1,5 +1,4 @@
 <?xml version="1.0" ?>
 <robot name="peg_board_assembly" xmlns:xacro="http://wiki.ros.org/xacro" >
-    <link name="world"/>
     <joint name="pb_world_joint" type="fixed">
         <parent link="world"/>
@@ -29,166 +28,3 @@
         </inertial>
     </link>
-    <joint name="pb_starter_joint" type="continuous">
-        <parent link="peg_board"/>
-        <child link="starter_gear"/>
-        <origin rpy="0 0 0" xyz="-0.375 0 0.125"/>
-        <axis xyz="0 0 1"/>
-        <limit effort="1500.0" velocity="10.0"/>
-        <dynamics damping="0.1" friction="0.01"/>
-    </joint>
-    <link name="starter_gear">
-        <visual>
-            <origin rpy="0 0 0" xyz="0 0 0"/>
-            <geometry>
-                <mesh filename="file://$(find sirgas_description)/meshes/Starter_Gear.stl" />
-            </geometry>
-            <material name="LightGrey">
-                <color rgba="0.7 0.7 0.7 1.0" />
-            </material>
-        </visual>
-        <collision>
-            <origin rpy="0 0 0" xyz="0 0 0"/>
-            <geometry>
-                <mesh filename="file://$(find sirgas_description)/meshes/Starter_Gear.stl" />
-            </geometry>
-        </collision>
-        <inertial>
-            <mass value="4.903"/>
-            <origin rpy="0 0 0" xyz="0 0 0"/>
-            <inertia ixx="0.0731301" ixy="0.0" ixz="0.0" iyx="0.0" iyy="0.073" iyz="0.0" izx="0.0" izy= "0.0" izz="0.14570353"/>
-        </inertial>
-    </link>
-    <joint name="pb_first_joint" type="continuous">
-        <parent link="peg_board"/>
-        <child link="first_gear"/>
-        <origin rpy="0 0 0" xyz="0 0 0.125"/>
-        <axis xyz="0 0 1"/>
-        <limit effort="1500.0" velocity="10.0"/>
-        <dynamics damping="0.1" friction="0.01"/>
-        <mimic joint="pb_starter_joint" multiplier="-1.76923" offset="0"/>
-    </joint>
-    <link name="first_gear">
-        <visual>
-            <origin rpy="0 0 0" xyz="0 0 0"/>
-            <geometry>
-                <mesh filename="file://$(find sirgas_description)/meshes/First_Gear.stl" />
-            </geometry>
-            <material name="LightGrey">
-                <color rgba="0.7 0.7 0.7 1.0" />
-            </material>
-        </visual>
-        <collision>
-            <origin rpy="0 0 0" xyz="0 0 0"/>
-            <geometry>
-                <mesh filename="file://$(find sirgas_description)/meshes/First_Gear.stl" />
-            </geometry>
-        </collision>
-        <inertial>
-            <mass value="1.409"/>
-            <origin rpy="0 0 0" xyz="0 0 0"/>
-            <inertia ixx="0.00615061" ixy="0.0" ixz="0.0" iyx="0.0" iyy="0.00615163" iyz="0.0" izx="0.0" izy= "0.0" izz="0.01209542"/>
-        </inertial>
-    </link>
-    <joint name="pb_second_joint" type="continuous">
-        <parent link="peg_board"/>
-        <child link="second_gear"/>
-        <origin rpy="0 0 0" xyz="0.25 0 0.125"/>
-        <axis xyz="0 0 1"/>
-        <limit effort="1500.0" velocity="10.0"/>
-        <dynamics damping="0.1" friction="0.01"/>
-        <mimic joint="pb_first_joint" multiplier="-1.0" offset="0"/>
-    </joint>
-    <link name="second_gear">
-        <visual>
-            <origin rpy="0 0 0" xyz="0 0 0"/>
-            <geometry>
-                <mesh filename="file://$(find sirgas_description)/meshes/Second_Gear.stl" />
-            </geometry>
-            <material name="LightGrey">
-                <color rgba="0.7 0.7 0.7 1.0" />
-            </material>
-        </visual>
-        <collision>
-            <origin rpy="0 0 0" xyz="0 0 0"/>
-            <geometry>
-                <mesh filename="file://$(find sirgas_description)/meshes/Second_Gear.stl" />
-            </geometry>
-        </collision>
-        <inertial>
-            <mass value="1.141"/>
-            <origin rpy="0 0 0" xyz="0 0 0.01359774"/>
-            <inertia ixx="0.00406128" ixy="0.0" ixz="0.0" iyx="0.0" iyy="0.00406281" iyz="0.0" izx="0.0" izy= "0.0" izz="0.00794573"/>
-        </inertial>
-    </link>
-    <joint name="pb_third_joint" type="continuous">
-        <parent link="peg_board"/>
-        <child link="third_gear"/>
-        <origin rpy="0 0 0" xyz="0.45 0 0.125"/>
-        <axis xyz="0 0 1"/>
-        <limit effort="1500.0" velocity="10.0"/>
-        <dynamics damping="0.1" friction="0.01"/>
-        <mimic joint="pb_second_joint" multiplier="-1.625" offset="0"/>
-    </joint>
-    <link name="third_gear">
-        <visual>
-            <origin rpy="0 0 0" xyz="0 0 0"/>
-            <geometry>
-                <mesh filename="file://$(find sirgas_description)/meshes/Third_Gear.stl" />
-            </geometry>
-            <material name="LightGrey">
-                <color rgba="0.7 0.7 0.7 1.0" />
-            </material>
-        </visual>
-        <collision>
-            <origin rpy="0 0 0" xyz="0 0 0"/>
-            <geometry>
-                <mesh filename="file://$(find sirgas_description)/meshes/Third_Gear.stl" />
-            </geometry>
-        </collision>
-        <inertial>
-            <mass value="0.538"/>
-            <origin rpy="0 0 0" xyz="0 0 0.01483255"/>
-            <inertia ixx="0.00095806" ixy="0.0" ixz="0.0" iyx="0.0" iyy="0.00095831" iyz="0.0" izx="0.0" izy= "0.0" izz="0.00180386"/>
-        </inertial>
-    </link>
-     <!-- ROS 2 Control configuration -->
-     <!-- Only the master joint (pb_starter_joint) gets command interfaces -->
-     <!-- Mimic joints only get state interfaces -->
-    <ros2_control name="peg_board_control" type="system">
-        <hardware>
-            <plugin>gz_ros2_control/GazeboSimSystem</plugin>
-        </hardware>
-        <joint name="pb_starter_joint">
-            <command_interface name="velocity">
-                <param name="min">-10</param>
-                <param name="max">10</param>
-            </command_interface>
-            <state_interface name="position"/>
-            <state_interface name="velocity"/>
-            <state_interface name="effort"/>
-        </joint>
-        <joint name="pb_first_joint">
-            <state_interface name="position"/>
-            <state_interface name="velocity"/>
-            <state_interface name="effort"/>
-        </joint>
-        <joint name="pb_second_joint">
-            <state_interface name="position"/>
-            <state_interface name="velocity"/>
-            <state_interface name="effort"/>
-        </joint>
-        <joint name="pb_third_joint">
-            <state_interface name="position"/>
-            <state_interface name="velocity"/>
-            <state_interface name="effort"/>
-        </joint>
-    </ros2_control>
-    <gazebo>
-        <plugin filename="libgz_ros2_control-system.so" name="gz_ros2_control::GazeboSimROS2ControlPlugin">
-            <parameters>$(find sirgas_description)/config/pba_controller.yaml</parameters>
-            <controller_manager_name>pba_controller_manager</controller_manager_name>
-            <robot_param>peg_board_assembly</robot_param>
-            <robot_param_node>/pba/robot_description</robot_param_node>
-        </plugin>
-    </gazebo>
 </robot>
