Commit message: Added script folder and script files to move the Panda and pba robots. Also had to update some urdf files, so both fingers on the gripper will move. Currently, only one figer moves

File: RBE594_ws/src/sirgas_description/urdf/panda_pba.urdf.xacro (robot description, xacro)
@@ -54,4 +54,9 @@
             <state_interface name="effort"/>
         </joint>
+        <joint name="panda_finger_joint2">
+            <state_interface name="position"/>
+            <state_interface name="velocity"/>
+            <state_interface name="effort"/>
+        </joint>
         <!-- PBA Robot -->
         <joint name="pb_starter_joint">

File: RBE594_ws/src/test_ws/config/panda_pba_robots.ros2_control.xacro (robot description, xacro)
@@ -72,4 +72,11 @@
                 <state_interface name="effort"/>
             </joint>
+            <joint name="panda_finger_joint2">
+              <state_interface name="position">
+                <param name="initial_value">${initial_positions['panda_finger_joint2']}</param>
+              </state_interface>
+              <state_interface name="velocity"/>
+              <state_interface name="effort"/>
+          </joint>
         </ros2_control>
     </xacro:macro>

Commit message: updating branch

File: RBE594_ws/src/sirgas_description/urdf/panda_pba.urdf.xacro (robot description, xacro)
@@ -9,4 +9,6 @@
     <!-- Import PBA Robot - directly include without macro call -->
     <xacro:include filename="$(find sirgas_description)/urdf/camera2.urdf.xacro" />
+    <!-- Import Cube for test grabbing -->
+    <xacro:include filename="$(find sirgas_description)/urdf/cube.urdf.xacro" />
     <ros2_control name="combined_controller" type="system">
         <hardware>

File: RBE594_ws/src/sirgas_description/urdf/pba2.urdf.xacro (robot description, xacro)
@@ -13,6 +13,6 @@
                 <mesh filename="file://$(find sirgas_description)/meshes/Peg_Board.stl" />
             </geometry>
-            <material name="LightGrey">
-                <color rgba="0.7 0.7 0.7 1.0" />
+            <material name="White">
+                <color rgba="1.0 1.0 1.0 1.0" />
             </material>
         </visual>
@@ -43,6 +43,6 @@
                 <mesh filename="file://$(find sirgas_description)/meshes/Starter_Gear.stl" />
             </geometry>
-            <material name="LightGrey">
-                <color rgba="0.7 0.7 0.7 1.0" />
+            <material name="DarkGrey">
+                <color rgba="0.25 0.25 0.25 1.0" />
             </material>
         </visual>
@@ -74,6 +74,6 @@
                 <mesh filename="file://$(find sirgas_description)/meshes/First_Gear.stl" />
             </geometry>
-            <material name="LightGrey">
-                <color rgba="0.7 0.7 0.7 1.0" />
+            <material name="DarkGrey">
+                <color rgba="0.25 0.25 0.25 1.0" />
             </material>
         </visual>
@@ -113,6 +113,6 @@
                 <mesh filename="file://$(find sirgas_description)/meshes/Second_Gear.stl" />
             </geometry>
-            <material name="LightGrey">
-                <color rgba="0.7 0.7 0.7 1.0" />
+            <material name="DarkGrey">
+                <color rgba="0.25 0.25 0.25 1.0" />
             </material>
         </visual>
@@ -144,6 +144,6 @@
                 <mesh filename="file://$(find sirgas_description)/meshes/Third_Gear.stl" />
             </geometry>
-            <material name="LightGrey">
-                <color rgba="0.7 0.7 0.7 1.0" />
+            <material name="DarkGrey">
+                <color rgba="0.25 0.25 0.25 1.0" />
             </material>
         </visual>
@@ -160,4 +160,141 @@
         </inertial>
     </link>
+    <!-- Liner Info -->
+    <link name="liner1">
+        <visual>
+            <origin rpy="0 0 0" xyz="0 0 0"/>
+            <geometry>
+                <box size="0.005 0.005 0.001"/>
+            </geometry>
+            <material name="Red">
+                <color rgba="1.0 0 0 1.0" />
+            </material>
+        </visual>
+    </link>
+    <joint name="liner1_pbs" type="fixed">
+        <parent link="peg_board"/>
+        <child link="liner1"/>
+        <origin rpy="0 0 0" xyz="-0.375 -0.02225 0.176"/>
+        <axis xyz="0 0 1"/>
+    </joint>
+    <link name="liner2">
+        <visual>
+            <origin rpy="0 0 0" xyz="0 0 0"/>
+            <geometry>
+                <box size="0.005 0.005 0.001"/>
+            </geometry>
+            <material name="Red">
+                <color rgba="1.0 0 0 1.0" />
+            </material>
+        </visual>
+    </link>
+    <joint name="liner2_pbs" type="fixed">
+        <parent link="starter_gear"/>
+        <child link="liner2"/>
+        <origin rpy="0 0 0" xyz="0.0 -0.028 0.051"/>
+        <axis xyz="0 0 1"/>
+    </joint>
+    <link name="liner3">
+        <visual>
+            <origin rpy="0 0 0" xyz="0 0 0"/>
+            <geometry>
+                <box size="0.005 0.005 0.001"/>
+            </geometry>
+            <material name="Red">
+                <color rgba="1.0 0 0 1.0" />
+            </material>
+        </visual>
+    </link>
+    <joint name="liner3_pbf" type="fixed">
+        <parent link="peg_board"/>
+        <child link="liner3"/>
+        <origin rpy="0 0 0" xyz="0.0 -0.02225 0.176"/>
+        <axis xyz="0 0 1"/>
+    </joint>
+    <link name="liner4">
+        <visual>
+            <origin rpy="0 0 0" xyz="0 0 0"/>
+            <geometry>
+                <box size="0.005 0.005 0.001"/>
+            </geometry>
+            <material name="Red">
+                <color rgba="1.0 0 0 1.0" />
+            </material>
+        </visual>
+    </link>
+    <joint name="liner4_pbf" type="fixed">
+        <parent link="first_gear"/>
+        <child link="liner4"/>
+        <origin rpy="0 0 0" xyz="0.0 -0.028 0.051"/>
+        <axis xyz="0 0 1"/>
+    </joint>
+    <link name="liner5">
+        <visual>
+            <origin rpy="0 0 0" xyz="0 0 0"/>
+            <geometry>
+                <box size="0.005 0.005 0.001"/>
+            </geometry>
+            <material name="Red">
+                <color rgba="1.0 0 0 1.0" />
+            </material>
+        </visual>
+    </link>
+    <joint name="liner5_pbf" type="fixed">
+        <parent link="peg_board"/>
+        <child link="liner5"/>
+        <origin rpy="0 0 0" xyz="0.25 -0.02225 0.176"/>
+        <axis xyz="0 0 1"/>
+    </joint>
+    <link name="liner6">
+        <visual>
+            <origin rpy="0 0 0" xyz="0 0 0"/>
+            <geometry>
+                <box size="0.005 0.005 0.001"/>
+            </geometry>
+            <material name="Red">
+                <color rgba="1.0 0 0 1.0" />
+            </material>
+        </visual>
+    </link>
+    <joint name="liner6_pb2" type="fixed">
+        <parent link="second_gear"/>
+        <child link="liner6"/>
+        <origin rpy="0 0 0" xyz="0.0 -0.028 0.051"/>
+        <axis xyz="0 0 1"/>
+    </joint>
+    <link name="liner7">
+        <visual>
+            <origin rpy="0 0 0" xyz="0 0 0"/>
+            <geometry>
+                <box size="0.005 0.005 0.001"/>
+            </geometry>
+            <material name="Red">
+                <color rgba="1.0 0 0 1.0" />
+            </material>
+        </visual>
+    </link>
+    <joint name="liner7_pbt" type="fixed">
+        <parent link="peg_board"/>
+        <child link="liner7"/>
+        <origin rpy="0 0 0" xyz="0.45 -0.02225 0.176"/>
+        <axis xyz="0 0 1"/>
+    </joint>
+    <link name="liner8">
+        <visual>
+            <origin rpy="0 0 0" xyz="0 0 0"/>
+            <geometry>
+                <box size="0.005 0.005 0.001"/>
+            </geometry>
+            <material name="Red">
+                <color rgba="1.0 0 0 1.0" />
+            </material>
+        </visual>
+    </link>
+    <joint name="liner8_pbt" type="fixed">
+        <parent link="third_gear"/>
+        <child link="liner8"/>
+        <origin rpy="0 0 0" xyz="0.0 -0.028 0.051"/>
+        <axis xyz="0 0 1"/>
+    </joint>
      <!-- ROS 2 Control configuration -->
      <!-- Only the master joint (pb_starter_joint) gets command interfaces -->

File: RBE594_ws/src/sirgas_description/urdf/ur20_pba.urdf.xacro (robot description, xacro)
@@ -4,5 +4,5 @@
     <link name="world"/>
     <!-- Import UR20 Robot - directly include without macro call -->
-    <xacro:include filename="$(find sirgas_description)/urdf/ur20_starter2.urdf.xacro" />
+    <xacro:include filename="$(find sirgas_description)/urdf/ur20_starter.urdf.xacro" />
     <!-- Import PBA Robot - directly include without macro call -->
     <xacro:include filename="$(find sirgas_description)/urdf/pba2.urdf.xacro" />

Commit message: updated files

File: RBE594_ws/src/sirgas_description/urdf/panda_pba.urdf.xacro (robot description, xacro)
@@ -62,5 +62,5 @@
         </joint>
         <!-- PBA Robot -->
-        <!-- <joint name="pb_starter_joint">
+        <joint name="pb_starter_joint">
             <command_interface name="velocity">
                 <param name="min">-10</param>
@@ -71,19 +71,4 @@
             <state_interface name="effort"/>
         </joint>
-        <joint name="pb_first_joint">
-            <state_interface name="position"/>
-            <state_interface name="velocity"/>
-            <state_interface name="effort"/>
-        </joint>
-        <joint name="pb_second_joint">
-            <state_interface name="position"/>
-            <state_interface name="velocity"/>
-            <state_interface name="effort"/>
-        </joint>
-        <joint name="pb_third_joint">
-            <state_interface name="position"/>
-            <state_interface name="velocity"/>
-            <state_interface name="effort"/>
-        </joint> -->
     </ros2_control>
     <gazebo>

File: RBE594_ws/src/sirgas_description/urdf/pba.urdf.xacro (robot description, xacro)
@@ -28,4 +28,34 @@
         </inertial>
     </link>
+    <joint name="pb_starter_joint" type="continuous">
+        <parent link="peg_board"/>
+        <child link="starter_gear"/>
+        <origin rpy="0 0 0" xyz="-0.375 0 0.125"/>
+        <axis xyz="0 0 1"/>
+        <limit effort="1500.0" velocity="10.0"/>
+        <dynamics damping="0.1" friction="0.01"/>
+    </joint>
+    <link name="starter_gear">
+        <visual>
+            <origin rpy="0 0 0" xyz="0 0 0"/>
+            <geometry>
+                <mesh filename="file://$(find sirgas_description)/meshes/Starter_Gear.stl" />
+            </geometry>
+            <material name="DarkGrey">
+                <color rgba="0.25 0.25 0.25 1.0" />
+            </material>
+        </visual>
+        <collision>
+            <origin rpy="0 0 0" xyz="0 0 0"/>
+            <geometry>
+                <mesh filename="file://$(find sirgas_description)/meshes/Starter_Gear.stl" />
+            </geometry>
+        </collision>
+        <inertial>
+            <mass value="4.903"/>
+            <origin rpy="0 0 0" xyz="0 0 0"/>
+            <inertia ixx="0.0731301" ixy="0.0" ixz="0.0" iyx="0.0" iyy="0.073" iyz="0.0" izx="0.0" izy= "0.0" izz="0.14570353"/>
+        </inertial>
+    </link>
     <!-- Liner Info -->
     <link name="liner1">
@@ -44,4 +74,21 @@
         <child link="liner1"/>
         <origin rpy="0 0 0" xyz="-0.375 -0.013125 0.226"/>
+        <axis xyz="0 0 1"/>
+    </joint>
+    <link name="liner2">
+        <visual>
+            <origin rpy="0 0 0" xyz="0 0 0"/>
+            <geometry>
+                <box size="0.005 0.005 0.001"/>
+            </geometry>
+            <material name="Red">
+                <color rgba="1.0 0 0 1.0" />
+            </material>
+        </visual>
+    </link>
+    <joint name="liner2_pbs" type="fixed">
+        <parent link="starter_gear"/>
+        <child link="liner2"/>
+        <origin rpy="0 0 0" xyz="0.0 -0.028 0.101"/>
         <axis xyz="0 0 1"/>
     </joint>
