Commit message: updated pba files

File: RBE594_ws/src/sirgas_description/urdf/pba.urdf.xacro (robot description, xacro)
@@ -66,5 +66,6 @@
         <limit effort="1500.0" lower="${-2*pi}" upper="${2*pi}" velocity="10.0"/>
         <dynamics damping="0" friction="0"/>
-    </joint>
+        <mimic joint="pb_starter_joint" multiplier="-1.76923" offset="0"/>
+        </joint>
     <link name="first_gear">
         <visual>
@@ -96,5 +97,6 @@
         <limit effort="1500.0" lower="${-2*pi}" upper="${2*pi}" velocity="10.0"/>
         <dynamics damping="0" friction="0"/>
-    </joint>
+        <mimic joint="pb_first_joint" multiplier="-1.0" offset="0"/>
+        </joint>
     <link name="second_gear">
         <visual>
@@ -126,5 +128,6 @@
         <limit effort="1500.0" lower="${-2*pi}" upper="${2*pi}" velocity="10.0"/>
         <dynamics damping="0" friction="0"/>
-    </joint>
+        <mimic joint="pb_second_joint" multiplier="-1.625" offset="0"/>
+        </joint>
     <link name="third_gear">
         <visual>
@@ -149,3 +152,35 @@
         </inertial>
     </link>
-</robot>
+    <xacro:macro name="peg_board_assembly_ros2_control">
+        <ros2_control name="GazeboSystem" type="system">
+            <hardware>
+                <plugin>gazebo_ros2_control/GazeboSystem</plugin>
+            </hardware>
+            <joint name="pb_starter_joint">
+                <command_interface name="velocity"/>
+                <state_interface name="position"/>
+                <state_interface name="velocity"/>
+                <param name="sim_hardware_interface">velocity_controllers/VelocityJointInterface</param>
+            </joint>
+            <joint name="pb_first_joint">
+                <command_interface name="velocity"/>
+                <state_interface name="position"/>
+                <state_interface name="velocity"/>
+                <param name="sim_hardware_interface">velocity_controllers/VelocityJointInterface</param>
+            </joint>
+            <joint name="pb_second_joint">
+                <command_interface name="velocity"/>
+                <state_interface name="position"/>
+                <state_interface name="velocity"/>
+                <param name="sim_hardware_interface">velocity_controllers/VelocityJointInterface</param>
+            </joint>
+            <joint name="pb_third_joint">
+                <command_interface name="velocity"/>
+                <state_interface name="position"/>
+                <state_interface name="velocity"/>
+                <param name="sim_hardware_interface">velocity_controllers/VelocityJointInterface</param>
+            </joint>
+        </ros2_control>
+    </xacro:macro>
+    <xacro:peg_board_assembly_ros2_control/>
+    </robot>

Commit message: Added .xml launch file and updated pba files.

File: RBE594_ws/src/sirgas_description/urdf/pba.urdf.xacro (robot description, xacro)
@@ -35,5 +35,5 @@
         <axis xyz="0 0 1"/>
         <limit effort="1500.0" lower="${-2*pi}" upper="${2*pi}" velocity="10.0"/>
-        <dynamics damping="0" friction="0"/>
+        <dynamics damping="0.1" friction="0.01"/>
     </joint>
     <link name="starter_gear">
@@ -65,7 +65,7 @@
         <axis xyz="0 0 1"/>
         <limit effort="1500.0" lower="${-2*pi}" upper="${2*pi}" velocity="10.0"/>
-        <dynamics damping="0" friction="0"/>
+        <dynamics damping="0.1" friction="0.01"/>
         <mimic joint="pb_starter_joint" multiplier="-1.76923" offset="0"/>
-        </joint>
+    </joint>
     <link name="first_gear">
         <visual>
@@ -96,7 +96,7 @@
         <axis xyz="0 0 1"/>
         <limit effort="1500.0" lower="${-2*pi}" upper="${2*pi}" velocity="10.0"/>
-        <dynamics damping="0" friction="0"/>
+        <dynamics damping="0.1" friction="0.01"/>
         <mimic joint="pb_first_joint" multiplier="-1.0" offset="0"/>
-        </joint>
+    </joint>
     <link name="second_gear">
         <visual>
@@ -127,7 +127,7 @@
         <axis xyz="0 0 1"/>
         <limit effort="1500.0" lower="${-2*pi}" upper="${2*pi}" velocity="10.0"/>
-        <dynamics damping="0" friction="0"/>
+        <dynamics damping="0.1" friction="0.01"/>
         <mimic joint="pb_second_joint" multiplier="-1.625" offset="0"/>
-        </joint>
+    </joint>
     <link name="third_gear">
         <visual>
@@ -152,35 +152,41 @@
         </inertial>
     </link>
-    <xacro:macro name="peg_board_assembly_ros2_control">
-        <ros2_control name="GazeboSystem" type="system">
-            <hardware>
-                <plugin>gazebo_ros2_control/GazeboSystem</plugin>
-            </hardware>
-            <joint name="pb_starter_joint">
-                <command_interface name="velocity"/>
-                <state_interface name="position"/>
-                <state_interface name="velocity"/>
-                <param name="sim_hardware_interface">velocity_controllers/VelocityJointInterface</param>
-            </joint>
-            <joint name="pb_first_joint">
-                <command_interface name="velocity"/>
-                <state_interface name="position"/>
-                <state_interface name="velocity"/>
-                <param name="sim_hardware_interface">velocity_controllers/VelocityJointInterface</param>
-            </joint>
-            <joint name="pb_second_joint">
-                <command_interface name="velocity"/>
-                <state_interface name="position"/>
-                <state_interface name="velocity"/>
-                <param name="sim_hardware_interface">velocity_controllers/VelocityJointInterface</param>
-            </joint>
-            <joint name="pb_third_joint">
-                <command_interface name="velocity"/>
-                <state_interface name="position"/>
-                <state_interface name="velocity"/>
-                <param name="sim_hardware_interface">velocity_controllers/VelocityJointInterface</param>
-            </joint>
-        </ros2_control>
-    </xacro:macro>
-    <xacro:peg_board_assembly_ros2_control/>
-    </robot>
+     <!-- ROS 2 Control configuration -->
+     <!-- Only the master joint (pb_starter_joint) gets command interfaces -->
+     <!-- Mimic joints only get state interfaces -->
+    <ros2_control name="peg_board_control" type="system">
+        <hardware>
+            <plugin>gz_ros2_control/GazeboSimSystem</plugin>
+        </hardware>
+        <joint name="pb_starter_joint">
+            <command_interface name="velocity">
+                <param name="min">-10</param>
+                <param name="max">10</param>
+            </command_interface>
+            <state_interface name="position"/>
+            <state_interface name="velocity"/>
+        </joint>
+        <joint name="pb_first_joint">
+            <!-- Only state interfaces for mimic joints -->
+            <state_interface name="position"/>
+            <state_interface name="velocity"/>
+        </joint>
+        <joint name="pb_second_joint">
+            <!-- Only state interfaces for mimic joints -->
+            <state_interface name="position"/>
+            <state_interface name="velocity"/>
+        </joint>
+        <joint name="pb_third_joint">
+            <!-- Only state interfaces for mimic joints -->
+            <state_interface name="position"/>
+            <state_interface name="velocity"/>
+        </joint>
+    </ros2_control>
+    <!-- Fixed Ignition Gazebo plugin for ROS 2 Control -->
+    <gazebo>
+        <plugin filename="libgz_ros2_control-system.so" name="gz_ros2_control::GazeboSimROS2ControlPlugin">
+            <parameters>$(find sirgas_description)/config/pba_controller.yaml</parameters>
+            <controller_manager_node_name>controller_manager</controller_manager_node_name>
+        </plugin>
+    </gazebo>
+</robot>

Commit message: updated pba files

File: RBE594_ws/src/sirgas_description/urdf/pba.urdf.xacro (robot description, xacro)
@@ -29,10 +29,10 @@
         </inertial>
     </link>
-    <joint name="pb_starter_joint" type="revolute">
+    <joint name="pb_starter_joint" type="continuous">
         <parent link="peg_board"/>
         <child link="starter_gear"/>
         <origin rpy="0 0 0" xyz="-0.375 0 0.125"/>
         <axis xyz="0 0 1"/>
-        <limit effort="1500.0" lower="${-2*pi}" upper="${2*pi}" velocity="10.0"/>
+        <limit effort="1500.0" velocity="10.0"/>
         <dynamics damping="0.1" friction="0.01"/>
     </joint>
@@ -59,10 +59,10 @@
         </inertial>
     </link>
-    <joint name="pb_first_joint" type="revolute">
+    <joint name="pb_first_joint" type="continuous">
         <parent link="peg_board"/>
         <child link="first_gear"/>
         <origin rpy="0 0 0" xyz="0 0 0.125"/>
         <axis xyz="0 0 1"/>
-        <limit effort="1500.0" lower="${-2*pi}" upper="${2*pi}" velocity="10.0"/>
+        <limit effort="1500.0" velocity="10.0"/>
         <dynamics damping="0.1" friction="0.01"/>
         <mimic joint="pb_starter_joint" multiplier="-1.76923" offset="0"/>
@@ -90,10 +90,10 @@
         </inertial>
     </link>
-    <joint name="pb_second_joint" type="revolute">
+    <joint name="pb_second_joint" type="continuous">
         <parent link="peg_board"/>
         <child link="second_gear"/>
         <origin rpy="0 0 0" xyz="0.25 0 0.125"/>
         <axis xyz="0 0 1"/>
-        <limit effort="1500.0" lower="${-2*pi}" upper="${2*pi}" velocity="10.0"/>
+        <limit effort="1500.0" velocity="10.0"/>
         <dynamics damping="0.1" friction="0.01"/>
         <mimic joint="pb_first_joint" multiplier="-1.0" offset="0"/>
@@ -121,10 +121,10 @@
         </inertial>
     </link>
-    <joint name="pb_third_joint" type="revolute">
+    <joint name="pb_third_joint" type="continuous">
         <parent link="peg_board"/>
         <child link="third_gear"/>
         <origin rpy="0 0 0" xyz="0.45 0 0.125"/>
         <axis xyz="0 0 1"/>
-        <limit effort="1500.0" lower="${-2*pi}" upper="${2*pi}" velocity="10.0"/>
+        <limit effort="1500.0" velocity="10.0"/>
         <dynamics damping="0.1" friction="0.01"/>
         <mimic joint="pb_second_joint" multiplier="-1.625" offset="0"/>
@@ -168,24 +168,19 @@
         </joint>
         <joint name="pb_first_joint">
-            <!-- Only state interfaces for mimic joints -->
             <state_interface name="position"/>
             <state_interface name="velocity"/>
         </joint>
         <joint name="pb_second_joint">
-            <!-- Only state interfaces for mimic joints -->
             <state_interface name="position"/>
             <state_interface name="velocity"/>
         </joint>
         <joint name="pb_third_joint">
-            <!-- Only state interfaces for mimic joints -->
             <state_interface name="position"/>
             <state_interface name="velocity"/>
         </joint>
     </ros2_control>
-    <!-- Fixed Ignition Gazebo plugin for ROS 2 Control -->
     <gazebo>
         <plugin filename="libgz_ros2_control-system.so" name="gz_ros2_control::GazeboSimROS2ControlPlugin">
             <parameters>$(find sirgas_description)/config/pba_controller.yaml</parameters>
-            <controller_manager_node_name>controller_manager</controller_manager_node_name>
         </plugin>
     </gazebo>

Commit message: uploading all new files

File: RBE594_ws/src/sirgas_description/urdf/pba.urdf.xacro (robot description, xacro)
@@ -188,4 +188,6 @@
             <parameters>$(find sirgas_description)/config/pba_controller.yaml</parameters>
             <controller_manager_name>pba_controller_manager</controller_manager_name>
+            <robot_param>peg_board_assembly</robot_param>
+            <robot_param_node>/pba/robot_description</robot_param_node>
         </plugin>
     </gazebo>

File: RBE594_ws/src/sirgas_description/urdf/ur20_starter.urdf.xacro (robot description, xacro)
@@ -81,5 +81,5 @@
      trajectory_port="$(arg trajectory_port)"
      >
-     <origin xyz="0.0 0.0 0.0" rpy="0 0 0" />  <!-- Position in world -->
+     <origin xyz="0.0 1.0 0.0" rpy="0 0 0" />  <!-- Position in world -->
    </xacro:ur_robot>
    <!-- Gazebo plugins - only add if this is the main robot in simulation -->
