Commit message: adding stuff

File: RBE594_ws/src/sirgas_description/urdf/pba.urdf.xacro (robot description, xacro)
@@ -1,194 +1,250 @@
-<?xml version="1.0" ?>
-<robot name="peg_board_assembly" xmlns:xacro="http://wiki.ros.org/xacro" >
-    <link name="world"/>
-    <joint name="pb_world_joint" type="fixed">
-        <parent link="world"/>
-        <child link="peg_board"/>
-        <origin rpy="0 0 0" xyz="0 0 0"/>
-    </joint>
-    <link name="peg_board">
-        <visual>
-            <origin rpy="0 0 0" xyz="0 0 0"/>
-            <geometry>
-                <mesh filename="file://$(find sirgas_description)/meshes/Peg_Board.stl" />
-            </geometry>
-            <material name="LightGrey">
-                <color rgba="0.7 0.7 0.7 1.0" />
-            </material>
-        </visual>
-        <collision>
-            <origin rpy="0 0 0" xyz="0 0 0"/>
-            <geometry>
-                <mesh filename="file://$(find sirgas_description)/meshes/Peg_Board.stl" />
-            </geometry>
-        </collision>
-        <inertial>
-            <mass value="170.447"/>
-            <origin rpy="0 0 0" xyz="0 0 0"/>
-            <inertia ixx="3.75895934" ixy="0.0" ixz="0.0" iyx="0.0" iyy="14.51416559" iyz="0.0" izx="-0.02634141" izy= "0.0" izz="17.74821744"/>
-        </inertial>
-    </link>
-    <joint name="pb_starter_joint" type="continuous">
-        <parent link="peg_board"/>
-        <child link="starter_gear"/>
-        <origin rpy="0 0 0" xyz="-0.375 0 0.125"/>
-        <axis xyz="0 0 1"/>
-        <limit effort="1500.0" velocity="10.0"/>
-        <dynamics damping="0.1" friction="0.01"/>
-    </joint>
-    <link name="starter_gear">
-        <visual>
-            <origin rpy="0 0 0" xyz="0 0 0"/>
-            <geometry>
-                <mesh filename="file://$(find sirgas_description)/meshes/Starter_Gear.stl" />
-            </geometry>
-            <material name="LightGrey">
-                <color rgba="0.7 0.7 0.7 1.0" />
-            </material>
-        </visual>
-        <collision>
-            <origin rpy="0 0 0" xyz="0 0 0"/>
-            <geometry>
-                <mesh filename="file://$(find sirgas_description)/meshes/Starter_Gear.stl" />
-            </geometry>
-        </collision>
-        <inertial>
-            <mass value="4.903"/>
-            <origin rpy="0 0 0" xyz="0 0 0"/>
-            <inertia ixx="0.0731301" ixy="0.0" ixz="0.0" iyx="0.0" iyy="0.073" iyz="0.0" izx="0.0" izy= "0.0" izz="0.14570353"/>
-        </inertial>
-    </link>
-    <joint name="pb_first_joint" type="continuous">
-        <parent link="peg_board"/>
-        <child link="first_gear"/>
-        <origin rpy="0 0 0" xyz="0 0 0.125"/>
-        <axis xyz="0 0 1"/>
-        <limit effort="1500.0" velocity="10.0"/>
-        <dynamics damping="0.1" friction="0.01"/>
-        <mimic joint="pb_starter_joint" multiplier="-1.76923" offset="0"/>
-    </joint>
-    <link name="first_gear">
-        <visual>
-            <origin rpy="0 0 0" xyz="0 0 0"/>
-            <geometry>
-                <mesh filename="file://$(find sirgas_description)/meshes/First_Gear.stl" />
-            </geometry>
-            <material name="LightGrey">
-                <color rgba="0.7 0.7 0.7 1.0" />
-            </material>
-        </visual>
-        <collision>
-            <origin rpy="0 0 0" xyz="0 0 0"/>
-            <geometry>
-                <mesh filename="file://$(find sirgas_description)/meshes/First_Gear.stl" />
-            </geometry>
-        </collision>
-        <inertial>
-            <mass value="1.409"/>
-            <origin rpy="0 0 0" xyz="0 0 0"/>
-            <inertia ixx="0.00615061" ixy="0.0" ixz="0.0" iyx="0.0" iyy="0.00615163" iyz="0.0" izx="0.0" izy= "0.0" izz="0.01209542"/>
-        </inertial>
-    </link>
-    <joint name="pb_second_joint" type="continuous">
-        <parent link="peg_board"/>
-        <child link="second_gear"/>
-        <origin rpy="0 0 0" xyz="0.25 0 0.125"/>
-        <axis xyz="0 0 1"/>
-        <limit effort="1500.0" velocity="10.0"/>
-        <dynamics damping="0.1" friction="0.01"/>
-        <mimic joint="pb_first_joint" multiplier="-1.0" offset="0"/>
-    </joint>
-    <link name="second_gear">
-        <visual>
-            <origin rpy="0 0 0" xyz="0 0 0"/>
-            <geometry>
-                <mesh filename="file://$(find sirgas_description)/meshes/Second_Gear.stl" />
-            </geometry>
-            <material name="LightGrey">
-                <color rgba="0.7 0.7 0.7 1.0" />
-            </material>
-        </visual>
-        <collision>
-            <origin rpy="0 0 0" xyz="0 0 0"/>
-            <geometry>
-                <mesh filename="file://$(find sirgas_description)/meshes/Second_Gear.stl" />
-            </geometry>
-        </collision>
-        <inertial>
-            <mass value="1.141"/>
-            <origin rpy="0 0 0" xyz="0 0 0.01359774"/>
-            <inertia ixx="0.00406128" ixy="0.0" ixz="0.0" iyx="0.0" iyy="0.00406281" iyz="0.0" izx="0.0" izy= "0.0" izz="0.00794573"/>
-        </inertial>
-    </link>
-    <joint name="pb_third_joint" type="continuous">
-        <parent link="peg_board"/>
-        <child link="third_gear"/>
-        <origin rpy="0 0 0" xyz="0.45 0 0.125"/>
-        <axis xyz="0 0 1"/>
-        <limit effort="1500.0" velocity="10.0"/>
-        <dynamics damping="0.1" friction="0.01"/>
-        <mimic joint="pb_second_joint" multiplier="-1.625" offset="0"/>
-    </joint>
-    <link name="third_gear">
-        <visual>
-            <origin rpy="0 0 0" xyz="0 0 0"/>
-            <geometry>
-                <mesh filename="file://$(find sirgas_description)/meshes/Third_Gear.stl" />
-            </geometry>
-            <material name="LightGrey">
-                <color rgba="0.7 0.7 0.7 1.0" />
-            </material>
-        </visual>
-        <collision>
-            <origin rpy="0 0 0" xyz="0 0 0"/>
-            <geometry>
-                <mesh filename="file://$(find sirgas_description)/meshes/Third_Gear.stl" />
-            </geometry>
-        </collision>
-        <inertial>
-            <mass value="0.538"/>
-            <origin rpy="0 0 0" xyz="0 0 0.01483255"/>
-            <inertia ixx="0.00095806" ixy="0.0" ixz="0.0" iyx="0.0" iyy="0.00095831" iyz="0.0" izx="0.0" izy= "0.0" izz="0.00180386"/>
-        </inertial>
-    </link>
-     <!-- ROS 2 Control configuration -->
-     <!-- Only the master joint (pb_starter_joint) gets command interfaces -->
-     <!-- Mimic joints only get state interfaces -->
-    <ros2_control name="peg_board_control" type="system">
-        <hardware>
-            <plugin>gz_ros2_control/GazeboSimSystem</plugin>
-        </hardware>
-        <joint name="pb_starter_joint">
-            <command_interface name="velocity">
-                <param name="min">-10</param>
-                <param name="max">10</param>
-            </command_interface>
-            <state_interface name="position"/>
-            <state_interface name="velocity"/>
-            <state_interface name="effort"/>
-        </joint>
-        <joint name="pb_first_joint">
-            <state_interface name="position"/>
-            <state_interface name="velocity"/>
-            <state_interface name="effort"/>
-        </joint>
-        <joint name="pb_second_joint">
-            <state_interface name="position"/>
-            <state_interface name="velocity"/>
-            <state_interface name="effort"/>
-        </joint>
-        <joint name="pb_third_joint">
-            <state_interface name="position"/>
-            <state_interface name="velocity"/>
-            <state_interface name="effort"/>
-        </joint>
-    </ros2_control>
-    <gazebo>
-        <plugin filename="libgz_ros2_control-system.so" name="gz_ros2_control::GazeboSimROS2ControlPlugin">
-            <parameters>$(find sirgas_description)/config/pba_controller.yaml</parameters>
-            <controller_manager_name>pba_controller_manager</controller_manager_name>
-            <robot_param>peg_board_assembly</robot_param>
-            <robot_param_node>/pba/robot_description</robot_param_node>
-        </plugin>
-    </gazebo>
+<?xml version="1.0"?>
+<robot name="peg_board_assembly" xmlns:xacro="http://wiki.ros.org/xacro">
+  <xacro:include filename="$(find sirgas_description)/urdf/inc/apriltag_card.xacro"/>
+  <link name="world"/>
+  <joint name="pb_world_joint" type="fixed">
+    <parent link="world"/>
+    <child link="peg_board"/>
+    <origin xyz="0 0 0" rpy="0 0 0"/>
+  </joint>
+  <link name="peg_board">
+    <visual>
+      <origin xyz="0 0 0" rpy="0 0 0"/>
+      <geometry>
+        <mesh filename="file://$(find sirgas_description)/meshes/Peg_Board.stl"/>
+      </geometry>
+      <material name="LightGrey">
+        <color rgba="0.7 0.7 0.7 1.0"/>
+      </material>
+    </visual>
+    <collision>
+      <origin xyz="0 0 0" rpy="0 0 0"/>
+      <geometry>
+        <mesh filename="file://$(find sirgas_description)/meshes/Peg_Board.stl"/>
+      </geometry>
+    </collision>
+    <inertial>
+      <mass value="170.447"/>
+      <origin xyz="0 0 0" rpy="0 0 0"/>
+      <inertia
+        ixx="3.75895934"
+        ixy="0.0"
+        ixz="0.0"
+        iyx="0.0"
+        iyy="14.51416559"
+        iyz="0.0"
+        izx="-0.02634141"
+        izy="0.0"
+        izz="17.74821744"/>
+    </inertial>
+  </link>
+  <joint name="pb_starter_joint" type="continuous">
+    <parent link="peg_board"/>
+    <child link="starter_gear"/>
+    <origin xyz="-0.375 0 0.125" rpy="0 0 0"/>
+    <axis xyz="0 0 1"/>
+    <limit effort="1500.0" velocity="10.0"/>
+    <dynamics damping="0.1" friction="0.01"/>
+  </joint>
+  <link name="starter_gear">
+    <visual>
+      <origin xyz="0 0 0" rpy="0 0 0"/>
+      <geometry>
+        <mesh filename="file://$(find sirgas_description)/meshes/Starter_Gear.stl"/>
+      </geometry>
+      <material name="LightGrey">
+        <color rgba="0.7 0.7 0.7 1.0"/>
+      </material>
+    </visual>
+    <collision>
+      <origin xyz="0 0 0" rpy="0 0 0"/>
+      <geometry>
+        <mesh filename="file://$(find sirgas_description)/meshes/Starter_Gear.stl"/>
+      </geometry>
+    </collision>
+    <inertial>
+      <mass value="4.903"/>
+      <origin xyz="0 0 0" rpy="0 0 0"/>
+      <inertia
+        ixx="0.0731301"
+        ixy="0.0"
+        ixz="0.0"
+        iyx="0.0"
+        iyy="0.073"
+        iyz="0.0"
+        izx="0.0"
+        izy="0.0"
+        izz="0.14570353"/>
+    </inertial>
+  </link>
+  <joint name="pb_first_joint" type="continuous">
+    <parent link="peg_board"/>
+    <child link="first_gear"/>
+    <origin xyz="0 0 0.125" rpy="0 0 0"/>
+    <axis xyz="0 0 1"/>
+    <limit effort="1500.0" velocity="10.0"/>
+    <dynamics damping="0.1" friction="0.01"/>
+    <mimic joint="pb_starter_joint" multiplier="-1.76923" offset="0"/>
+  </joint>
+  <link name="first_gear">
+    <visual>
+      <origin xyz="0 0 0" rpy="0 0 0"/>
+      <geometry>
+        <mesh filename="file://$(find sirgas_description)/meshes/First_Gear.stl"/>
+      </geometry>
+      <material name="LightGrey">
+        <color rgba="0.7 0.7 0.7 1.0"/>
+      </material>
+    </visual>
+    <collision>
+      <origin xyz="0 0 0" rpy="0 0 0"/>
+      <geometry>
+        <mesh filename="file://$(find sirgas_description)/meshes/First_Gear.stl"/>
+      </geometry>
+    </collision>
+    <inertial>
+      <mass value="1.409"/>
+      <origin xyz="0 0 0" rpy="0 0 0"/>
+      <inertia
+        ixx="0.00615061"
+        ixy="0.0"
+        ixz="0.0"
+        iyx="0.0"
+        iyy="0.00615163"
+        iyz="0.0"
+        izx="0.0"
+        izy="0.0"
+        izz="0.01209542"/>
+    </inertial>
+  </link>
+  <xacro:attach_apriltag_card
+    parent_link="first_gear"
+    link_name="first_gear_apriltag"
+    tag_size="0.05"
+    tag_thickness="0.0015"
+    xyz="0 0 0.02"
+    rpy="0 0 0"
+    material_script_uri_1="model://Apriltag36_11_00000/materials/scripts"
+    material_script_uri_2="model://Apriltag36_11_00000/materials/textures"
+    material_name="Apriltag/Tag36_11_00000"/>
+  <joint name="pb_second_joint" type="continuous">
+    <parent link="peg_board"/>
+    <child link="second_gear"/>
+    <origin xyz="0.25 0 0.125" rpy="0 0 0"/>
+    <axis xyz="0 0 1"/>
+    <limit effort="1500.0" velocity="10.0"/>
+    <dynamics damping="0.1" friction="0.01"/>
+    <mimic joint="pb_first_joint" multiplier="-1.0" offset="0"/>
+  </joint>
+  <link name="second_gear">
+    <visual>
+      <origin xyz="0 0 0" rpy="0 0 0"/>
+      <geometry>
+        <mesh filename="file://$(find sirgas_description)/meshes/Second_Gear.stl"/>
+      </geometry>
+      <material name="LightGrey">
+        <color rgba="0.7 0.7 0.7 1.0"/>
+      </material>
+    </visual>
+    <collision>
+      <origin xyz="0 0 0" rpy="0 0 0"/>
+      <geometry>
+        <mesh filename="file://$(find sirgas_description)/meshes/Second_Gear.stl"/>
+      </geometry>
+    </collision>
+    <inertial>
+      <mass value="1.141"/>
+      <origin xyz="0 0 0.01359774" rpy="0 0 0"/>
+      <inertia
+        ixx="0.00406128"
+        ixy="0.0"
+        ixz="0.0"
+        iyx="0.0"
+        iyy="0.00406281"
+        iyz="0.0"
+        izx="0.0"
+        izy="0.0"
+        izz="0.00794573"/>
+    </inertial>
+  </link>
+  <joint name="pb_third_joint" type="continuous">
+    <parent link="peg_board"/>
+    <child link="third_gear"/>
+    <origin xyz="0.45 0 0.125" rpy="0 0 0"/>
+    <axis xyz="0 0 1"/>
+    <limit effort="1500.0" velocity="10.0"/>
+    <dynamics damping="0.1" friction="0.01"/>
+    <mimic joint="pb_second_joint" multiplier="-1.625" offset="0"/>
+  </joint>
+  <link name="third_gear">
+    <visual>
+      <origin xyz="0 0 0" rpy="0 0 0"/>
+      <geometry>
+        <mesh filename="file://$(find sirgas_description)/meshes/Third_Gear.stl"/>
+      </geometry>
+      <material name="LightGrey">
+        <color rgba="0.7 0.7 0.7 1.0"/>
+      </material>
+    </visual>
+    <collision>
+      <origin xyz="0 0 0" rpy="0 0 0"/>
+      <geometry>
+        <mesh filename="file://$(find sirgas_description)/meshes/Third_Gear.stl"/>
+      </geometry>
+    </collision>
+    <inertial>
+      <mass value="0.538"/>
+      <origin xyz="0 0 0.01483255" rpy="0 0 0"/>
+      <inertia
+        ixx="0.00095806"
+        ixy="0.0"
+        ixz="0.0"
+        iyx="0.0"
+        iyy="0.00095831"
+        iyz="0.0"
+        izx="0.0"
+        izy="0.0"
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
File: RBE594_ws/src/sirgas_description/urdf/pba2.urdf.xacro (robot description, xacro)
@@ -89,4 +89,14 @@
         </inertial>
     </link>
+    <xacro:attach_apriltag_card
+    parent_link="first_gear"
+    link_name="first_gear_apriltag"
+    tag_size="0.05"
+    tag_thickness="0.0015"
+    xyz="0 0 0.02"
+    rpy="0 0 0"
+    material_script_uri_1="model://Apriltag36_11_00000/materials/scripts"
+    material_script_uri_2="model://Apriltag36_11_00000/materials/textures"
+    material_name="Apriltag/Tag36_11_00000"/>
     <joint name="pb_second_joint" type="continuous">
         <parent link="peg_board"/>

File: RBE594_ws/src/sirgas_description/urdf/ur20_pba.urdf.xacro (robot description, xacro)
@@ -3,4 +3,5 @@
     <!-- World fixed link -->
     <link name="world"/>
+    <xacro:include filename="$(find sirgas_description)/urdf/inc/apriltag_card.xacro"/>
     <!-- Import UR20 Robot - directly include without macro call -->
     <xacro:include filename="$(find sirgas_description)/urdf/ur20_starter2.urdf.xacro" />

Commit message: Added Cartesian Path Planner and attached other gears to peg board to prevent them from moving around withough being touched

File: RBE594_ws/src/sirgas_description/urdf/pba.urdf.xacro (robot description, xacro)
@@ -58,4 +58,64 @@
         </inertial>
     </link>
+    <joint name="pb_second_joint" type="continuous">
+        <parent link="peg_board"/>
+        <child link="second_gear"/>
+        <origin rpy="0 0 0" xyz="0.25 0 0.125"/>
+        <axis xyz="0 0 1"/>
+        <limit effort="1500.0" velocity="10.0"/>
+        <dynamics damping="0.1" friction="0.01"/>
+    </joint>
+    <link name="second_gear">
+        <visual>
+            <origin rpy="0 0 0" xyz="0 0 0"/>
+            <geometry>
+                <mesh filename="file://$(find sirgas_description)/meshes/Second_Gear.stl" />
+            </geometry>
+            <material name="DarkGrey">
+                <color rgba="0.25 0.25 0.25 1.0" />
+            </material>
+        </visual>
+        <collision>
+            <origin rpy="0 0 0" xyz="0 0 0"/>
+            <geometry>
+                <mesh filename="file://$(find sirgas_description)/meshes/Second_Gear.stl" />
+            </geometry>
+        </collision>
+        <inertial>
+            <mass value="1.141"/>
+            <origin rpy="0 0 0" xyz="0 0 0.01359774"/>
+            <inertia ixx="0.00406128" ixy="0.0" ixz="0.0" iyx="0.0" iyy="0.00406281" iyz="0.0" izx="0.0" izy= "0.0" izz="0.00794573"/>
+        </inertial>
+    </link>
+    <joint name="pb_third_joint" type="continuous">
+        <parent link="peg_board"/>
+        <child link="third_gear"/>
+        <origin rpy="0 0 0" xyz="0.45 0 0.125"/>
+        <axis xyz="0 0 1"/>
+        <limit effort="1500.0" velocity="10.0"/>
+        <dynamics damping="0.1" friction="0.01"/>
+    </joint>
+    <link name="third_gear">
+        <visual>
+            <origin rpy="0 0 0" xyz="0 0 0"/>
+            <geometry>
+                <mesh filename="file://$(find sirgas_description)/meshes/Third_Gear.stl" />
+            </geometry>
+            <material name="DarkGrey">
+                <color rgba="0.25 0.25 0.25 1.0" />
+            </material>
+        </visual>
+        <collision>
+            <origin rpy="0 0 0" xyz="0 0 0"/>
+            <geometry>
+                <mesh filename="file://$(find sirgas_description)/meshes/Third_Gear.stl" />
+            </geometry>
+        </collision>
+        <inertial>
+            <mass value="0.538"/>
+            <origin rpy="0 0 0" xyz="0 0 0.01483255"/>
+            <inertia ixx="0.00095806" ixy="0.0" ixz="0.0" iyx="0.0" iyy="0.00095831" iyz="0.0" izx="0.0" izy= "0.0" izz="0.00180386"/>
+        </inertial>
+    </link>
     <!-- Liner Info -->
     <link name="liner1">
@@ -127,4 +187,21 @@
         <axis xyz="0 0 1"/>
     </joint>
+    <link name="liner6">
+        <visual>
+            <origin rpy="0 0 0" xyz="0 0 0"/>
+            <geometry>
+                <box size="0.005 0.005 0.001"/>
+            </geometry>
+            <material name="Red">
+                <color rgba="1.0 0 0 1.0" />
+            </material>
+        </visual>
+    </link>
+    <joint name="liner6_pb2" type="fixed">
+        <parent link="second_gear"/>
+        <child link="liner6"/>
+        <origin rpy="0 0 0" xyz="0.0 -0.028 0.051"/>
+        <axis xyz="0 0 1"/>
+    </joint>
     <link name="liner7">
         <visual>
@@ -144,3 +221,20 @@
         <axis xyz="0 0 1"/>
     </joint>
+    <link name="liner8">
+        <visual>
+            <origin rpy="0 0 0" xyz="0 0 0"/>
+            <geometry>
+                <box size="0.005 0.005 0.001"/>
+            </geometry>
+            <material name="Red">
+                <color rgba="1.0 0 0 1.0" />
+            </material>
+        </visual>
+    </link>
+    <joint name="liner8_pbt" type="fixed">
+        <parent link="third_gear"/>
+        <child link="liner8"/>
+        <origin rpy="0 0 0" xyz="0.0 -0.028 0.051"/>
+        <axis xyz="0 0 1"/>
+    </joint>
 </robot>

Commit message: Updated mesh files.

File: RBE594_ws/src/sirgas_description/urdf/pba.urdf.xacro (robot description, xacro)
@@ -155,7 +155,7 @@
     <link name="liner3">
         <visual>
-            <origin rpy="0 0 0" xyz="0 0 0"/>
-            <geometry>
-                <box size="0.005 0.005 0.001"/>
+            <origin rpy="0 0 0" xyz="0 .0125 0"/>
+            <geometry>
+                <box size="0.005 0.025 0.001"/>
             </geometry>
             <material name="Green">
@@ -176,6 +176,6 @@
                 <box size="0.005 0.005 0.001"/>
             </geometry>
-            <material name="Blue">
-                <color rgba="0 0 1.0 1.0" />
+            <material name="Red">
+                <color rgba="1.0 0 0 1.0" />
             </material>
         </visual>
