Commit message: Updated grab_gear and mesh files

File: RBE594_ws/src/sirgas_description/urdf/first_gear.urdf.xacro (robot description, xacro)
@@ -35,5 +35,5 @@
         <parent link="first_gear"/>
         <child link="liner4"/>
-        <origin rpy="0 0 0" xyz="0.0 -0.028 0.051"/>
+        <origin rpy="0 0 0" xyz="0.0 -0.028 0.0655"/>
         <axis xyz="0 0 1"/>
     </joint>

File: RBE594_ws/src/sirgas_description/urdf/panda.urdf.xacro (robot description, xacro)
@@ -280,5 +280,5 @@
         <origin rpy="0 0 0" xyz="0 0 0.0584" />
         <axis xyz="0 1 0" />
-        <limit effort="20" lower="0.0" upper="0.04" velocity="0.2" />
+        <limit effort="200" lower="0.0" upper="0.04" velocity="0.2" />
         <dynamics damping="0.3" />
     </joint>
@@ -288,5 +288,5 @@
         <origin rpy="0 0 0" xyz="0 0 0.0584" />
         <axis xyz="0 -1 0" />
-        <limit effort="20" lower="0.0" upper="0.04" velocity="0.2" />
+        <limit effort="200" lower="0.0" upper="0.04" velocity="0.2" />
         <mimic joint="panda_finger_joint1" />
         <dynamics damping="0.3" />

File: RBE594_ws/src/sirgas_description/urdf/pba.urdf.xacro (robot description, xacro)
@@ -28,3 +28,72 @@
         </inertial>
     </link>
+    <!-- Liner Info -->
+    <link name="liner1">
+        <visual>
+            <origin rpy="0 0 0" xyz="0 0 0"/>
+            <geometry>
+                <box size="0.005 0.005 0.001"/>
+            </geometry>
+            <material name="Red">
+                <color rgba="1.0 0 0 1.0" />
+            </material>
+        </visual>
+    </link>
+    <joint name="liner1_pbs" type="fixed">
+        <parent link="peg_board"/>
+        <child link="liner1"/>
+        <origin rpy="0 0 0" xyz="-0.375 -0.02225 0.191"/>
+        <axis xyz="0 0 1"/>
+    </joint>
+    <link name="liner3">
+        <visual>
+            <origin rpy="0 0 0" xyz="0 0 0"/>
+            <geometry>
+                <box size="0.005 0.005 0.001"/>
+            </geometry>
+            <material name="Red">
+                <color rgba="1.0 0 0 1.0" />
+            </material>
+        </visual>
+    </link>
+    <joint name="liner3_pbf" type="fixed">
+        <parent link="peg_board"/>
+        <child link="liner3"/>
+        <origin rpy="0 0 0" xyz="0.0 -0.02225 0.1905"/>
+        <axis xyz="0 0 1"/>
+    </joint>
+    <link name="liner5">
+        <visual>
+            <origin rpy="0 0 0" xyz="0 0 0"/>
+            <geometry>
+                <box size="0.005 0.005 0.001"/>
+            </geometry>
+            <material name="Red">
+                <color rgba="1.0 0 0 1.0" />
+            </material>
+        </visual>
+    </link>
+    <joint name="liner5_pbf" type="fixed">
+        <parent link="peg_board"/>
+        <child link="liner5"/>
+        <origin rpy="0 0 0" xyz="0.25 -0.02225 0.1905"/>
+        <axis xyz="0 0 1"/>
+    </joint>
+    <link name="liner7">
+        <visual>
+            <origin rpy="0 0 0" xyz="0 0 0"/>
+            <geometry>
+                <box size="0.005 0.005 0.001"/>
+            </geometry>
+            <material name="Red">
+                <color rgba="1.0 0 0 1.0" />
+            </material>
+        </visual>
+    </link>
+    <joint name="liner7_pbt" type="fixed">
+        <parent link="peg_board"/>
+        <child link="liner7"/>
+        <origin rpy="0 0 0" xyz="0.45 -0.02225 0.1905"/>
+        <axis xyz="0 0 1"/>
+    </joint>
 </robot>

File: RBE594_ws/src/sirgas_description/urdf/second_gear.urdf.xacro (robot description, xacro)
@@ -38,5 +38,5 @@
         <parent link="second_gear"/>
         <child link="liner6"/>
-        <origin rpy="0 0 0" xyz="0.0 -0.028 0.051"/>
+        <origin rpy="0 0 0" xyz="0.0 -0.028 0.0655"/>
         <axis xyz="0 0 1"/>
     </joint>

File: RBE594_ws/src/sirgas_description/urdf/starter_gear.urdf.xacro (robot description, xacro)
@@ -38,5 +38,5 @@
         <parent link="starter_gear"/>
         <child link="liner2"/>
-        <origin rpy="0 0 0" xyz="0.0 -0.028 0.051"/>
+        <origin rpy="0 0 0" xyz="0.0 -0.028 0.0655"/>
         <axis xyz="0 0 1"/>
     </joint>

File: RBE594_ws/src/sirgas_description/urdf/third_gear.urdf.xacro (robot description, xacro)
@@ -38,5 +38,5 @@
         <parent link="third_gear"/>
         <child link="liner8"/>
-        <origin rpy="0 0 0" xyz="0.0 -0.028 0.051"/>
+        <origin rpy="0 0 0" xyz="0.0 -0.028 0.0655"/>
         <axis xyz="0 0 1"/>
     </joint>

Commit message: updated files

File: RBE594_ws/src/sirgas_description/urdf/first_gear.urdf.xacro (robot description, xacro)
@@ -1,5 +1,5 @@
 <?xml version="1.0" ?>
 <robot name="first_gear" xmlns:xacro="http://wiki.ros.org/xacro" >
-    <xacro:include filename="$(find sirgas_description)/urdf/inc/apriltag_card.xacro"/>
+    <!-- <xacro:include filename="$(find sirgas_description)/urdf/inc/apriltag_card.xacro"/> -->
     <link name="first_gear">
         <visual>
@@ -24,5 +24,5 @@
         </inertial>
     </link>
-    <xacro:attach_apriltag_card
+    <!-- <xacro:attach_apriltag_card
         parent_link="first_gear"
         tag_size=".5"
@@ -31,9 +31,9 @@
         rpy="0 3.0 0"
         link_name="first_gear_apriltag"
-    />
+    /> -->
     <joint name="liner4_pbf" type="fixed">
         <parent link="first_gear"/>
         <child link="liner4"/>
-        <origin rpy="0 0 0" xyz="0.0 -0.028 0.0655"/>
+        <origin rpy="0 0 0" xyz="0.0 -0.028 0.101"/>
         <axis xyz="0 0 1"/>
     </joint>
@@ -45,6 +45,6 @@
                 <box size="0.005 0.005 0.001"/>
             </geometry>
-            <material name="Red">
-                <color rgba="1.0 0 0 1.0" />
+            <material name="Green">
+                <color rgba="0 1.0 0 1.0" />
             </material>
         </visual>

File: RBE594_ws/src/sirgas_description/urdf/panda.urdf.xacro (robot description, xacro)
@@ -280,5 +280,5 @@
         <origin rpy="0 0 0" xyz="0 0 0.0584" />
         <axis xyz="0 1 0" />
-        <limit effort="200" lower="0.0" upper="0.04" velocity="0.2" />
+        <limit effort="2000" lower="0.0" upper="0.04" velocity="0.2" />
         <dynamics damping="0.3" />
     </joint>
@@ -288,5 +288,5 @@
         <origin rpy="0 0 0" xyz="0 0 0.0584" />
         <axis xyz="0 -1 0" />
-        <limit effort="200" lower="0.0" upper="0.04" velocity="0.2" />
+        <limit effort="2000" lower="0.0" upper="0.04" velocity="0.2" />
         <mimic joint="panda_finger_joint1" />
         <dynamics damping="0.3" />

File: RBE594_ws/src/sirgas_description/urdf/pba.urdf.xacro (robot description, xacro)
@@ -43,5 +43,5 @@
         <parent link="peg_board"/>
         <child link="liner1"/>
-        <origin rpy="0 0 0" xyz="-0.375 -0.02225 0.191"/>
+        <origin rpy="0 0 0" xyz="-0.375 -0.013125 0.226"/>
         <axis xyz="0 0 1"/>
     </joint>
@@ -52,6 +52,6 @@
                 <box size="0.005 0.005 0.001"/>
             </geometry>
-            <material name="Red">
-                <color rgba="1.0 0 0 1.0" />
+            <material name="Green">
+                <color rgba="0 1.0 0 1.0" />
             </material>
         </visual>
@@ -60,5 +60,5 @@
         <parent link="peg_board"/>
         <child link="liner3"/>
-        <origin rpy="0 0 0" xyz="0.0 -0.02225 0.1905"/>
+        <origin rpy="0 0 0" xyz="0.0 -0.013125 0.226"/>
         <axis xyz="0 0 1"/>
     </joint>
@@ -69,6 +69,6 @@
                 <box size="0.005 0.005 0.001"/>
             </geometry>
-            <material name="Red">
-                <color rgba="1.0 0 0 1.0" />
+            <material name="Blue">
+                <color rgba="0 0 1.0 1.0" />
             </material>
         </visual>
@@ -77,5 +77,5 @@
         <parent link="peg_board"/>
         <child link="liner5"/>
-        <origin rpy="0 0 0" xyz="0.25 -0.02225 0.1905"/>
+        <origin rpy="0 0 0" xyz="0.25 -0.013125 0.226"/>
         <axis xyz="0 0 1"/>
     </joint>
@@ -86,6 +86,6 @@
                 <box size="0.005 0.005 0.001"/>
             </geometry>
-            <material name="Red">
-                <color rgba="1.0 0 0 1.0" />
+            <material name="Purple">
+                <color rgba="1.0 0 1.0 1.0" />
             </material>
         </visual>
@@ -94,5 +94,5 @@
         <parent link="peg_board"/>
         <child link="liner7"/>
-        <origin rpy="0 0 0" xyz="0.45 -0.02225 0.1905"/>
+        <origin rpy="0 0 0" xyz="0.45 -0.013125 0.226"/>
         <axis xyz="0 0 1"/>
     </joint>

File: RBE594_ws/src/sirgas_description/urdf/second_gear.urdf.xacro (robot description, xacro)
@@ -30,6 +30,6 @@
                 <box size="0.005 0.005 0.001"/>
             </geometry>
-            <material name="Red">
-                <color rgba="1.0 0 0 1.0" />
+            <material name="Blue">
+                <color rgba="0 0 1.0 1.0" />
             </material>
         </visual>
@@ -38,5 +38,5 @@
         <parent link="second_gear"/>
         <child link="liner6"/>
-        <origin rpy="0 0 0" xyz="0.0 -0.028 0.0655"/>
+        <origin rpy="0 0 0" xyz="0.0 -0.028 0.101"/>
         <axis xyz="0 0 1"/>
     </joint>

File: RBE594_ws/src/sirgas_description/urdf/starter_gear.urdf.xacro (robot description, xacro)
@@ -38,5 +38,5 @@
         <parent link="starter_gear"/>
         <child link="liner2"/>
-        <origin rpy="0 0 0" xyz="0.0 -0.028 0.0655"/>
+        <origin rpy="0 0 0" xyz="0.0 -0.028 0.101"/>
         <axis xyz="0 0 1"/>
     </joint>

File: RBE594_ws/src/sirgas_description/urdf/third_gear.urdf.xacro (robot description, xacro)
@@ -30,6 +30,6 @@
                 <box size="0.005 0.005 0.001"/>
             </geometry>
-            <material name="Red">
-                <color rgba="1.0 0 0 1.0" />
+            <material name="Purple">
+                <color rgba="1.0 0 1.0 1.0" />
             </material>
         </visual>
@@ -38,5 +38,5 @@
         <parent link="third_gear"/>
         <child link="liner8"/>
-        <origin rpy="0 0 0" xyz="0.0 -0.028 0.0655"/>
+        <origin rpy="0 0 0" xyz="0.0 -0.028 0.101"/>
         <axis xyz="0 0 1"/>
     </joint>

Commit message: added topics for publishing the useful axis

File: RBE594_ws/src/sirgas_description/urdf/first_gear.urdf.xacro (robot description, xacro)
@@ -1,5 +1,5 @@
 <?xml version="1.0" ?>
 <robot name="first_gear" xmlns:xacro="http://wiki.ros.org/xacro" >
-    <!-- <xacro:include filename="$(find sirgas_description)/urdf/inc/apriltag_card.xacro"/> -->
+    <xacro:include filename="$(find sirgas_description)/urdf/inc/apriltag_card.xacro"/>
     <link name="first_gear">
         <visual>
@@ -24,12 +24,12 @@
         </inertial>
     </link>
-    <!-- <xacro:attach_apriltag_card
+    <xacro:attach_apriltag_card
         parent_link="first_gear"
-        tag_size=".5"
-        tag_thickness="0.00001"
-        xyz="0 .06 1.0"
-        rpy="0 3.0 0"
-        link_name="first_gear_apriltag"
-    /> -->
+        tag_size="0.02"
+        extra_len="0.03"
+        tag_thickness="0.0005"
+        xyz="0 0.075 0.025"
+        rpy="0 3.14 .15"
+        link_name="first_gear_apriltag"/>
     <joint name="liner4_pbf" type="fixed">
         <parent link="first_gear"/>

File: RBE594_ws/src/sirgas_description/urdf/pba.urdf.xacro (robot description, xacro)
@@ -155,7 +155,7 @@
     <link name="liner3">
         <visual>
-            <origin rpy="0 0 0" xyz="0 0 0"/>
-            <geometry>
-                <box size="0.005 0.005 0.001"/>
+            <origin rpy="0 0 0" xyz="0 .0125 0"/>
+            <geometry>
+                <box size="0.005 0.025 0.001"/>
             </geometry>
             <material name="Green">

Commit message: workingon stuff

File: RBE594_ws/src/sirgas_description/urdf/first_gear.urdf.xacro (robot description, xacro)
@@ -30,7 +30,7 @@
         tag_thickness="0.0005"
         xyz="0 0.075 0.025"
-        rpy="0 3.14 .15"
+        rpy="0 3.14 0"
         link_name="first_gear_apriltag"/>
-    <joint name="liner4_pbf" type="fixed">
+    <!-- <joint name="liner4_pbf" type="fixed">
         <parent link="first_gear"/>
         <child link="liner4"/>
@@ -38,5 +38,4 @@
         <axis xyz="0 0 1"/>
     </joint>
-    <!-- Liner Info -->
     <link name="liner4">
         <visual>
@@ -49,4 +48,4 @@
             </material>
         </visual>
-    </link>
+    </link> -->
 </robot>

File: RBE594_ws/src/sirgas_description/urdf/pba.urdf.xacro (robot description, xacro)
@@ -157,5 +157,5 @@
             <origin rpy="0 0 0" xyz="0 .0125 0"/>
             <geometry>
-                <box size="0.005 0.025 0.001"/>
+                <box size="0.010 0.025 0.001"/>
             </geometry>
             <material name="Green">
@@ -176,6 +176,6 @@
                 <box size="0.005 0.005 0.001"/>
             </geometry>
-            <material name="Red">
-                <color rgba="1.0 0 0 1.0" />
+            <material name="Blue">
+                <color rgba="0 0 1.0 1.0" />
             </material>
         </visual>

Commit message: added more testing functions

File: RBE594_ws/src/sirgas_description/urdf/first_gear.urdf.xacro (robot description, xacro)
@@ -30,6 +30,7 @@
         tag_thickness="0.0005"
         xyz="0 0.075 0.025"
-        rpy="0 3.14 .15"
+        rpy="0 3.14 0"
         link_name="first_gear_apriltag"/>
+<!--
     <joint name="liner4_pbf" type="fixed">
         <parent link="first_gear"/>
@@ -38,5 +39,4 @@
         <axis xyz="0 0 1"/>
     </joint>
-    <!-- Liner Info -->
     <link name="liner4">
         <visual>
@@ -49,4 +49,4 @@
             </material>
         </visual>
-    </link>
+    </link> -->
 </robot>

Commit message: Edited rotate hand function

File: RBE594_ws/src/sirgas_description/urdf/first_gear.urdf.xacro (robot description, xacro)
@@ -19,5 +19,5 @@
         </collision>
         <inertial>
-            <mass value="1.409"/>
+            <mass value="0.409"/>
             <origin rpy="0 0 0" xyz="0 0 0"/>
             <inertia ixx="0.00615061" ixy="0.0" ixz="0.0" iyx="0.0" iyy="0.00615163" iyz="0.0" izx="0.0" izy= "0.0" izz="0.01209542"/>

Commit message: Updated files

File: RBE594_ws/src/sirgas_description/urdf/first_gear.urdf.xacro (robot description, xacro)
@@ -26,5 +26,5 @@
     <xacro:attach_apriltag_card
         parent_link="first_gear"
-        tag_size="0.02"
+        tag_size="0.01"
         extra_len="0.03"
         tag_thickness="0.0005"

File: RBE594_ws/src/sirgas_description/urdf/pba.urdf.xacro (robot description, xacro)
@@ -133,5 +133,5 @@
         <parent link="peg_board"/>
         <child link="liner1"/>
-        <origin rpy="0 0 0" xyz="-0.375 -0.013125 0.226"/>
+        <origin rpy="0 0 0" xyz="-0.375 -0.01 0.226"/>
         <axis xyz="0 0 1"/>
     </joint>
@@ -155,5 +155,5 @@
     <link name="liner3">
         <visual>
-            <origin rpy="0 0 0" xyz="0 .0125 0"/>
+            <origin rpy="0 0 0" xyz="0 0 0"/>
             <geometry>
                 <box size="0.005 0.025 0.001"/>
@@ -167,5 +167,5 @@
         <parent link="peg_board"/>
         <child link="liner3"/>
-        <origin rpy="0 0 0" xyz="0.0 -0.013125 0.226"/>
+        <origin rpy="0 0 0" xyz="0.0 0 0.226"/>
         <axis xyz="0 0 1"/>
     </joint>
@@ -184,5 +184,5 @@
         <parent link="peg_board"/>
         <child link="liner5"/>
-        <origin rpy="0 0 0" xyz="0.25 -0.013125 0.226"/>
+        <origin rpy="0 0 0" xyz="0.25 -0.01 0.226"/>
         <axis xyz="0 0 1"/>
     </joint>
@@ -201,5 +201,5 @@
         <parent link="second_gear"/>
         <child link="liner6"/>
-        <origin rpy="0 0 0" xyz="0.0 -0.028 0.051"/>
+        <origin rpy="0 0 0" xyz="0.0 -0.028 0.101"/>
         <axis xyz="0 0 1"/>
     </joint>
@@ -218,5 +218,5 @@
         <parent link="peg_board"/>
         <child link="liner7"/>
-        <origin rpy="0 0 0" xyz="0.45 -0.013125 0.226"/>
+        <origin rpy="0 0 0" xyz="0.45 -0.01 0.226"/>
         <axis xyz="0 0 1"/>
     </joint>
@@ -235,5 +235,5 @@
         <parent link="third_gear"/>
         <child link="liner8"/>
-        <origin rpy="0 0 0" xyz="0.0 -0.028 0.051"/>
+        <origin rpy="0 0 0" xyz="0.0 -0.028 0.101"/>
         <axis xyz="0 0 1"/>
     </joint>
