Commit message: fixed camera with move it, apriltag still broken

File: RBE594_ws/src/sirgas_description/urdf/inc/apriltag_card.xacro (robot description, xacro)
@@ -1,17 +1,18 @@
 <?xml version="1.0"?>
 <robot xmlns:xacro="http://wiki.ros.org/xacro">
+  <!-- Attach a thin AprilTag "card" to parent_link -->
   <xacro:macro name="attach_apriltag_card" params="
       parent_link
       tag_size:=0.05
       tag_thickness:=0.001
-      xyz:='0 0 0'
+      xyz:='0 0 0.02'
       rpy:='0 0 0'
       link_name:='${parent_link}_apriltag'
       mass:=0.01
-      material_script_uri_1:='model://Apriltag36_11_00000/materials/scripts'
-      material_script_uri_2:='model://Apriltag36_11_00000/materials/textures'
-      material_name:='Apriltag/Tag36_11_00000'
-    ">
+      texture_path:='package://sirgas_description/meshes/Apriltag36_11_00000/materials/textures/tag36_11_00000.png'
+      add_back_visual:=true
+      back_epsilon:=0.0005">
     <link name="${link_name}">
+      <!-- front face -->
       <visual>
         <origin xyz="${xyz}" rpy="${rpy}"/>
@@ -19,12 +20,20 @@
           <box size="${tag_size} ${tag_size} ${tag_thickness}"/>
         </geometry>
-        <material name="${material_name}">
-          <script>
-            <uri>${material_script_uri_1}</uri>
-            <uri>${material_script_uri_2}</uri>
-            <name>${material_name}</name>
-          </script>
+        <material name="${link_name}_front_tex">
+          <texture filename="${texture_path}"/>
         </material>
       </visual>
+      <!-- optional back face for RViz (flipped 180 deg around Y) -->
+      <xacro:if value="${add_back_visual}">
+        <visual>
+          <origin xyz="${xyz}" rpy="0 3.141592653589793 0"/>
+          <geometry>
+            <box size="${tag_size} ${tag_size} ${tag_thickness}"/>
+          </geometry>
+          <material name="${link_name}_back_tex">
+            <texture filename="${texture_path}"/>
+          </material>
+        </visual>
+      </xacro:if>
       <collision>
         <origin xyz="${xyz}" rpy="${rpy}"/>
@@ -36,8 +45,9 @@
         <origin xyz="0 0 0" rpy="0 0 0"/>
         <mass value="${mass}"/>
-        <inertia ixx="${mass*((tag_size*tag_size + tag_thickness*tag_thickness)/12.0)}"
-                 iyy="${mass*((tag_size*tag_size + tag_thickness*tag_thickness)/12.0)}"
-                 izz="${mass*((tag_size*tag_size + tag_size*tag_size)/12.0)}"
-                 ixy="0" ixz="0" iyz="0"/>
+        <inertia
+          ixx="${mass*((tag_size*tag_size + tag_thickness*tag_thickness)/12.0)}"
+          iyy="${mass*((tag_size*tag_size + tag_thickness*tag_thickness)/12.0)}"
+          izz="${mass*((tag_size*tag_size + tag_size*tag_size)/12.0)}"
+          ixy="0" ixz="0" iyz="0"/>
       </inertial>
     </link>
@@ -47,4 +57,20 @@
       <origin xyz="0 0 0" rpy="0 0 0"/>
     </joint>
+    <!-- Gazebo rendering: visible from both sides + small emissive + PBR albedo -->
+    <gazebo reference="${link_name}">
+      <material>
+        <double_sided>1</double_sided>
+        <ambient>0.6 0.6 0.6 1</ambient>
+        <diffuse>1 1 1 1</diffuse>
+        <emissive>0.05 0.05 0.05 1</emissive>
+        <pbr>
+          <metal>
+            <albedo_map>package://sirgas_description/meshes/Apriltag36_11_00000/materials/textures/tag36_11_00000.png</albedo_map>
+            <roughness>1.0</roughness>
+            <metalness>0.0</metalness>
+          </metal>
+        </pbr>
+      </material>
+    </gazebo>
   </xacro:macro>
 </robot>

File: RBE594_ws/src/sirgas_description/urdf/pba2.urdf.xacro (robot description, xacro)
@@ -1,4 +1,5 @@
 <?xml version="1.0" ?>
 <robot name="peg_board_assembly" xmlns:xacro="http://wiki.ros.org/xacro" >
+    <xacro:include filename="$(find sirgas_description)/urdf/inc/apriltag_card.xacro"/>
     <joint name="pb_world_joint" type="fixed">
         <parent link="world"/>
@@ -89,4 +90,12 @@
         </inertial>
     </link>
+    <xacro:attach_apriltag_card
+    parent_link="first_gear"
+    tag_size=".5"
+    tag_thickness="0.002"
+    xyz="0 .06 1.0"
+    rpy="0 3.14 0"
+    link_name="first_gear_apriltag"
+    />
     <joint name="pb_second_joint" type="continuous">
         <parent link="peg_board"/>

Commit message: Add apriltag helpers and gear alignment sim

File: RBE594_ws/src/sirgas_description/urdf/inc/apriltag_card.xacro (robot description, xacro)
@@ -4,5 +4,6 @@
   <xacro:macro name="attach_apriltag_card" params="
       parent_link
-      tag_size:=0.05
+      tag_size:=0.02
+      extra_len:=0.03
       tag_thickness:=0.001
       xyz:='0 0 0.02'
@@ -11,6 +12,9 @@
       mass:=0.01
       texture_path:='package://sirgas_description/meshes/Apriltag36_11_00000/materials/textures/tag36_11_00000.png'
-      add_back_visual:=true
+      add_back_visual:=false
       back_epsilon:=0.0005">
+    <xacro:property name="size_x" value="${tag_size}"/>
+    <xacro:property name="size_y" value="${tag_size + extra_len}"/>
+    <xacro:property name="size_z" value="${tag_thickness}"/>
     <link name="${link_name}">
       <!-- front face -->
@@ -18,5 +22,5 @@
         <origin xyz="${xyz}" rpy="${rpy}"/>
         <geometry>
-          <box size="${tag_size} ${tag_size} ${tag_thickness}"/>
+          <box size="${size_x} ${size_y} ${size_z}"/>
         </geometry>
         <material name="${link_name}_front_tex">
@@ -39,16 +43,15 @@
         <origin xyz="${xyz}" rpy="${rpy}"/>
         <geometry>
-          <box size="${tag_size} ${tag_size} ${tag_thickness}"/>
+           <box size="${size_x} ${size_y} ${size_z}"/>
         </geometry>
       </collision>
       <inertial>
-        <origin xyz="0 0 0" rpy="0 0 0"/>
-        <mass value="${mass}"/>
-        <inertia
-          ixx="${mass*((tag_size*tag_size + tag_thickness*tag_thickness)/12.0)}"
-          iyy="${mass*((tag_size*tag_size + tag_thickness*tag_thickness)/12.0)}"
-          izz="${mass*((tag_size*tag_size + tag_size*tag_size)/12.0)}"
-          ixy="0" ixz="0" iyz="0"/>
-      </inertial>
+          <origin xyz="0 0 0" rpy="0 0 0"/>
+          <mass value="${mass}"/>
+          <xacro:property name="Ixx" value="${mass*((size_y*size_y + size_z*size_z)/12.0)}"/>
+          <xacro:property name="Iyy" value="${mass*((size_x*size_x + size_z*size_z)/12.0)}"/>
+          <xacro:property name="Izz" value="${mass*((size_x*size_x + size_y*size_y)/12.0)}"/>
+          <inertia ixx="${Ixx}" iyy="${Iyy}" izz="${Izz}" ixy="0" ixz="0" iyz="0"/>
+        </inertial>
     </link>
     <joint name="${link_name}_fixed" type="fixed">
@@ -57,5 +60,4 @@
       <origin xyz="0 0 0" rpy="0 0 0"/>
     </joint>
-    <!-- Gazebo rendering: visible from both sides + small emissive + PBR albedo -->
     <gazebo reference="${link_name}">
       <material>

Commit message: Add apriltag helpers and gear alignment sim

File: RBE594_ws/src/sirgas_description/urdf/inc/apriltag_card.xacro (robot description, xacro)
@@ -4,5 +4,6 @@
   <xacro:macro name="attach_apriltag_card" params="
       parent_link
-      tag_size:=0.05
+      tag_size:=0.02
+      extra_len:=0.03
       tag_thickness:=0.001
       xyz:='0 0 0.02'
@@ -13,4 +14,7 @@
       add_back_visual:=false
       back_epsilon:=0.0005">
+    <xacro:property name="size_x" value="${tag_size}"/>
+    <xacro:property name="size_y" value="${tag_size + extra_len}"/>
+    <xacro:property name="size_z" value="${tag_thickness}"/>
     <link name="${link_name}">
       <!-- front face -->
@@ -18,5 +22,5 @@
         <origin xyz="${xyz}" rpy="${rpy}"/>
         <geometry>
-          <box size="${tag_size} ${tag_size} ${tag_thickness}"/>
+          <box size="${size_x} ${size_y} ${size_z}"/>
         </geometry>
         <material name="${link_name}_front_tex">
@@ -39,16 +43,15 @@
         <origin xyz="${xyz}" rpy="${rpy}"/>
         <geometry>
-          <box size="${tag_size} ${tag_size} ${tag_thickness}"/>
+           <box size="${size_x} ${size_y} ${size_z}"/>
         </geometry>
       </collision>
       <inertial>
-        <origin xyz="0 0 0" rpy="0 0 0"/>
-        <mass value="${mass}"/>
-        <inertia
-          ixx="${mass*((tag_size*tag_size + tag_thickness*tag_thickness)/12.0)}"
-          iyy="${mass*((tag_size*tag_size + tag_thickness*tag_thickness)/12.0)}"
-          izz="${mass*((tag_size*tag_size + tag_size*tag_size)/12.0)}"
-          ixy="0" ixz="0" iyz="0"/>
-      </inertial>
+          <origin xyz="0 0 0" rpy="0 0 0"/>
+          <mass value="${mass}"/>
+          <xacro:property name="Ixx" value="${mass*((size_y*size_y + size_z*size_z)/12.0)}"/>
+          <xacro:property name="Iyy" value="${mass*((size_x*size_x + size_z*size_z)/12.0)}"/>
+          <xacro:property name="Izz" value="${mass*((size_x*size_x + size_y*size_y)/12.0)}"/>
+          <inertia ixx="${Ixx}" iyy="${Iyy}" izz="${Izz}" ixy="0" ixz="0" iyz="0"/>
+        </inertial>
     </link>
     <joint name="${link_name}_fixed" type="fixed">
